File: hardware/CatStick.sch (KiCad schematic (older format))
At the start: 98 parts, among them J3 SMA, J4 U.FL, J5 USB_B_Micro, J6 Conn_02x05_Odd_Even, SW1 SW_Push, U2 ATSAMR34J18B, U2 CC1352R1F3RGZR, U3 SKY13373-460LF, Y1 48MHz, Y1 ABS05-32.768KHZ-9-T, Y2 32.768kHz

Commit message: Change to SAMD21E and SX1262 LoRa
Parts:
- removed C1: 10uF, Capacitor_SMD:C_0402_1005Metric, symbol Device:C
- removed C10, C11, C13, C14, C15, C2, C3, C35, C4, C5, C6, C8, C9: 100nF, Capacitor_SMD:C_0201_0603Metric, symbol Device:C
- removed C12, C33: 4.7pF, Capacitor_SMD:C_0201_0603Metric, symbol Device:C
- removed C16: DNM, Capacitor_SMD:C_0201_0603Metric, symbol Device:C_Small
- removed C17: 18pF, Capacitor_SMD:C_0201_0603Metric, symbol Device:C_Small
- removed C18: 3.9pF, Capacitor_SMD:C_0201_0603Metric, symbol Device:C_Small
- removed C19, C21: 3.3pF, Capacitor_SMD:C_0201_0603Metric, symbol Device:C_Small
- removed C20: 5.6pF, Capacitor_SMD:C_0201_0603Metric, symbol Device:C_Small
- removed C34: 1nF, Capacitor_SMD:C_0201_0603Metric, symbol Device:C
- removed C36, C37: 10pF, Capacitor_SMD:C_0201_0603Metric, symbol Device:C
- removed C7: 33pF, Capacitor_SMD:C_0201_0603Metric, symbol Device:C
- removed FB1: BLM15AG121SN1D, Inductor_SMD:L_0402_1005Metric, symbol Device:Ferrite_Bead
- removed JP1: RFSW_VCC_SLCT, Pads_Jumpers:JP_NO_NC, symbol Jumper:SolderJumper_3_Bridged12
- removed L10, L11, L4, L5: 10nH, Inductor_SMD:L_0201_0603Metric, symbol Device:L_Small
- removed L3: 2.2nH, Inductor_SMD:L_0402_1005Metric, symbol Device:L_Small
- removed L8: 33nH, Inductor_SMD:L_0201_0603Metric, symbol Device:L_Small
- removed L9: 11nH, Inductor_SMD:L_0201_0603Metric, symbol Device:L_Small
- removed R1: 100K, Resistor_SMD:R_0402_1005Metric, symbol Device:R
- removed U2: ATSAMR34J18B, gkl_housings_bga:TFBGA-64_6.0x6.0mm_Layout8x8_P0.65mm, symbol CatStick-rescue:ATSAMR34J18BT-TinyLoraModule-Symbol-Lib-TLM-v1-rescue-TLM-v1_2-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
- removed U3: SKY13373-460LF, gkl_housings_qfn:QFN-12-1EP_3x3mm_P0.5mm_EP1.65x1.65mm, symbol CatStick-rescue:SKY13373-460LF-TinyLoraModule-Symbol-Lib-TLM-v1-rescue-TLM-v1_2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
- removed XC1: TYETBCSANF-32.000000, gkl_time:Oscilator_2.5x2.0, symbol CatStick-rescue:TYETBCSANF-32.000000-TinyLoraModule-Symbol-Lib-TLM-v1-rescue-TL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
- removed Y1: ABS05-32.768KHZ-9-T, gkl_time:ABS05_32.768KHz Crystal, symbol Device:Crystal
- added SW2: RST, symbol Switch:SW_Push
- added U6: PE4259 RF Switch, Package_TO_SOT_SMD:SOT-363_SC-70-6, symbol RF_Switch:MASWSS0115
- added U7: ATSAMD21E18A-A, Package_QFP:TQFP-32_7x7mm_P0.8mm, symbol MCU_Microchip_SAMD:ATSAMD21E18A-A
- added U8: SX1262IMLTRT, QFN50P400X400X100-25N, symbol SX1262IMLTRT:SX1262IMLTRT
- added Y3: 32Mhz_10pF_10ppm, symbol Device:Crystal_GND24
- C22: value 47pF -> 0.1uF; footprint Capacitor_SMD:C_0201_0603Metric -> (none); Mfg 250R05L470GV4T -> (none)
- C23: value 2.7pF -> 0.1uF; footprint Capacitor_SMD:C_0201_0603Metric -> (none); Mfg GJM0335C1E2R7BB01E -> (none)
- C24, C26: value DNM -> 0.1uF; footprint Capacitor_SMD:C_0201_0603Metric -> (none); Mfg 1 -> (none)
- C25: value 4.7nF -> 18pF; footprint Capacitor_SMD:C_0201_0603Metric -> (none); Mfg GRM033R71A472KA01D -> (none)
- C27: value DNM -> 18pF; footprint Capacitor_SMD:C_0201_0603Metric -> (none); Mfg 1 -> (none)
- C28: value 22pF -> 0.1uF; footprint Capacitor_SMD:C_0201_0603Metric -> (none); Mfg 250R05L220GV4T -> (none)
- C29: value 3.9pF -> 100nF; footprint Capacitor_SMD:C_0201_0603Metric -> (none); Mfg GRM0335C1H3R9BA01D -> (none)
- C30: value 8.2pF -> 470nF; footprint Capacitor_SMD:C_0201_0603Metric -> (none); Mfg 250R05L8R2CV4T -> (none)
- C31: value 5.6pF -> 0.1uF; footprint Capacitor_SMD:C_0201_0603Metric -> (none); Mfg GRM0335C1E5R6BA01D -> (none)
- C32: value 3.3pF -> 47pF; footprint Capacitor_SMD:C_0201_0603Metric -> (none); Mfg 250R05L3R3BV4T -> (none)
- L6: value 33nH -> 15uH; footprint Inductor_SMD:L_0201_0603Metric -> (none); Mfg L-05B33NJV6T -> (none)
- L7: value 10nH -> 47nH; footprint Inductor_SMD:L_0201_0603Metric -> (none); Mfg MLK0603L10NJT000 -> (none)
- gave numbers to parts that had none: 9
- renumbered C13 to C1, C23 to C10, C2 to C11, C3 to C12, C4 to C13, C5 to C14, C7 to C15, C8 to C16, C10 to C17, C6 to C18, C9 to C19, C15 to C2, C11 to C20, C22 to C21, C34 to C4, C35 to C5, C33 to C6, C21 to C8, C1 to C9, J3 to J1, J4 to J2, J5 to J3, J6 to J4, L2 to L1, L16 to L2, L6 to L3, L1 to L4, L9 to L5, R1 to R2, U2 to U1, Y2 to Y1, Y1 to Y2
Connections:
- net labels added: +3.3V, ANT_SW, BUSY, CIPO, COPI, DIO1, DIO3, Dx, NSS, RESET_CC, RESET_SX, SCK, SW_RFI, SW_RFO
- net labels removed: ANT_PAD, BAND_SEL, PA14, PA15, PA18, PA19, PA_BOOST, RFI_HF, RFO_HF, SWDCLK, TCXO_PWR, TXRX_RF, TXRX_RFM, VDD, VDDA, VR_PA, XIN32, XOUT32, XTA
- wire segments 449 -> 306
- no-connect marks 40 -> 29
Other:
- note added: "I2C:"
- note added: "SAMD21E"
- note added: "SPI: LORA\nSERCOM3"
- note added: "SWD FOR SAMD21E"
- note added: "UART with\nRTS and CTS\nSERCOM0"
- note removed: "0"
- note removed: "1"
- note removed: "1.8-3.5 V"
- note removed: "1.8-3.6 V"
- note removed: "32MHz"
- note removed: "868 MHz Tx Matching"
- note removed: "868/915 MHz Rx Matching"
- note removed: "915 MHz Tx Matching"
- note removed: "IMPORTADO DE PINGUINO SAMR34 KICAD, SIN CAMBIOS"
- note removed: "NOTA: CAMBIAR POR BALUN"
- note removed: "NOTA: CAMBIAR POR SWITCH"
- note removed: "NOTA: REVISION??"
- note removed: "PSU in Linear Mode"
- note removed: "RFC—>PA_BOOST"
- note removed: "RFC—>RFI_HF"
- note removed: "RFC—>RFO_HF"
- note removed: "RFSW State"
- note removed: "SAMR34"
- note removed: "SWD FOR SAMR34"
- note removed: "Shutdown"
- note removed: "V1"
- note removed: "V2"
- moved on the sheet: AE1, BT1, C1, C10, C11, C12, C13, C14, C15, C16, C17, C18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

Commit message: switch RF
Parts:
- removed U3: RFSW6062, QFN40P200X200X60-15N, symbol CatStick-rescue:RFSW6062SR-RFSW6062SR-CatStick-rescue
- added AE2: Antenna, cc1350:2450AT45A100, symbol Device:Antenna
- added C33, C34: 1nF, symbol Device:C_Small
- added C35, C36, C38, C39: 100pF, Capacitor_SMD:C_0603_1608Metric, symbol Device:C
- added C37, C40, C41: 100pF, Capacitor_SMD:C_0402_1005Metric, symbol Device:C
- added J6: SMA, Connector_Coaxial:SMA_Amphenol_132289_EdgeMount, symbol Connector:Conn_Coaxial
- added L8: DNM, Inductor_SMD:L_0402_1005Metric, symbol Device:L
- added R4, R5: 100R, symbol Device:R_Small
- added U3: RFSW8006QTR7, Package_DFN_QFN:DFN-8-1EP_2x2mm_P0.5mm_EP0.9x1.3mm, symbol electroniccats:RFSW8006QTR7
Connections:
- net labels added: CTF1, CTF2, CTF3, CTLoRa, LoRA_O
- wire segments 306 -> 341
- no-connect marks 29 -> 24
Other:
- moved on the sheet: AE1, BT1, C10, C24, C25, C27, C29, C30, C31, C32, C4, C5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

Commit message: addAntenna
Parts:
- removed AE1, AE2: Antenna, cc1350:2450AT45A100, symbol Device:Antenna
- removed C41: 100pF, Capacitor_SMD:C_0402_1005Metric, symbol Device:C
- removed J1, J6: SMA, Connector_Coaxial:SMA_Amphenol_132289_EdgeMount, symbol Connector:Conn_Coaxial
- removed L2, L8: DNM, Inductor_SMD:L_0402_1005Metric, symbol Device:L
- C4: value DNM -> 100pF
- C5, C6: value 100pF -> 3.3pF
- L1: value DNM -> 9.1nH
Connections:
- net CTLoRa is gone; now on net ANT_SW: R4.2, U7.27 (PA28)
- net Dx is gone; now on net CTF3: U7.17 (PA16)
- net CTF3: no longer U7.25 (PA27)
- net GND: now also C40.1, C5.2, C6.2; no longer C40.2, L1.2
- net RX_TX: now also C40.2
- net UBP_2_4_GHZ: no longer C4.2, C5.2
- net UBP_SUB-1_GHZ: now also C37.1; no longer C6.2, U5.4 (UBP_SUB-1_GHZ)
- net at C6.1: now also C4.2, L1.2; no longer L1.1
- net at C4.1: now also U6.5 (RFC); no longer J2.1 (In)
- net LORA_O: now reaches C5.1
- net LORA_O: now also C35.1, L1.1
- net ANT: now reaches C39.2
- net ANT: now also J2.1 (In)
- net at C37.2: now also U5.4 (UBP_SUB-1_GHZ); no longer C40.1
- removed net LoRA_O: C35.1, C37.1, U6.5 (RFC)
- net SCL: no longer names the net of U7.12 (PA09)
- net SDA: no longer names the net of U7.11 (PA08)
- no-connect marks 24 -> 27
Other:
- note added: "SX1262 AND RF SWITCH\n"
- moved on the sheet: BT1, C10, C24, C25, C27, C29, C30, C31, C32, C33, C34, C35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

Commit message: selectCapacitors
Parts:
- C1, C11, C13, C2: LCSC# (none) -> C1642; manf# (none) -> 0603CG120J500NT; provedor (none) -> LCSC
- C10, C12, C14, C15, C17, C19, C20, C21: LCSC# (none) -> C14663; manf# (none) -> CC0603KRX7R9BB104; provedor (none) -> LCSC
- C16, C18: LCSC# (none) -> C109447; manf# (none) -> CC0603MRX5R6BB226; provedor (none) -> LCSC
- C22, C23, C24, C26, C28, C31: footprint (none) -> Capacitor_SMD:C_0603_1608Metric; LCSC# (none) -> C42998; manf# (none) -> 0603F104M500NT; provedor (none) -> LCSC
- C25, C27: footprint (none) -> Capacitor_SMD:C_0603_1608Metric; LCSC# (none) -> C165734; manf# (none) -> 0603CG180F500NT; provedor (none) -> LCSC
- C29: footprint (none) -> Capacitor_SMD:C_0603_1608Metric; LCSC# (none) -> C14663; manf# (none) -> CC0603KRX7R9BB104; provedor (none) -> LCSC
- C3, C7: LCSC# (none) -> C376802; manf# (none) -> TCC0603COG7R5D500CT; provedor (none) -> LCSC
- C30: footprint (none) -> Capacitor_SMD:C_0603_1608Metric; LCSC# (none) -> C170149; MANUFACTURER (none) -> C170149; manf# (none) -> CL10A474KB8NNNC; provedor (none) -> LCSC
- C32: footprint (none) -> Capacitor_SMD:C_0603_1608Metric; LCSC# (none) -> C519486; manf# (none) -> CC0603FRNPO9BN470; provedor (none) -> LCSC
- C33, C34: footprint (none) -> Capacitor_SMD:C_0603_1608Metric; LCSC# (none) -> C1588; manf# (none) -> CL10B102KB8NNNC; provedor (none) -> LCSC
- C35, C36, C38, C39: LCSC# (none) -> C14858; manf# (none) -> CL10C101JB8NNNC; provedor (none) -> LCSC
- C37, C4, C40: footprint Capacitor_SMD:C_0402_1005Metric -> Capacitor_SMD:C_0603_1608Metric; LCSC# (none) -> C14858; manf# (none) -> CL10C101JB8NNNC; provedor (none) -> LCSC
- C5, C6: LCSC# (none) -> C162225; manf# (none) -> GRM1885C1H3R3CA01D; provedor (none) -> LCSC
- C8, C9: LCSC# (none) -> C108343; manf# (none) -> 0603F105M500NT; provedor (none) -> LCSC
- U3: PARTREV 772-RFSW8006QTR7 -> (none); manf# (none) -> 772-RFSW8006QTR7
