File: hardware/CatStick.sch (KiCad schematic (older format))
At the start: 78 parts, among them J2 Antenna, J4 Conn_02x05_Odd_Even, J5 Conn_01x04, P1 USB_C_Plug_USB2.0, Q1 DMN6140L, SW1 SW_Push, SW2 RST, U1 CC1352R1F3RGZR, U2 AP2112K-3.3, U3 RFSW8006QTR7, U4 0900FM15D0039, U5 0900PC15A0036, U6 PE4259 RF Switch, U7 ATSAMD21E18A-A, U8 SX1262IMLTRT, Y1 32.768kHz, Y2 48MHz, Y3 32Mhz_10pF_10ppm

Commit message: fixFootprint
Parts:
- added D?: LED, LED_SMD:LED_0603_1608Metric_Pad1.05x0.95mm_HandSolder, symbol Device:LED_Small
- added JP?: Jumper, symbol Jumper:Jumper_3_Bridged12
- added R?: 330, Resistor_SMD:R_0603_1608Metric_Pad0.98x0.95mm_HandSolder, symbol Device:R_Small
- SW2: footprint (none) -> Button_Switch_SMD:SW_SPST_TL3342
- U8: footprint QFN50P400X400X100-25N -> Package_DFN_QFN:QFN-24-1EP_4x4mm_P0.5mm_EP2.65x2.65mm
- Y2: footprint Crystal:Crystal_SMD_HC49-SD -> Crystal:Crystal_SMD_3225-4Pin_3.2x2.5mm; LCSC# C240990 -> C389928; manf# 49MD-48.000-20-20-20/A -> 7325-4800A1620-00
Connections:
- net labels added: DIO22, LED4
- wire segments 343 -> 352
- no-connect marks 24 -> 23
Other:
- note added: "LEDs\n\n\n"
- note removed: "LEDs SAMD21E\n\n"
- moved on the sheet: C34, D1, D2, D3, R10, R5, R8, R9

Commit message: fixPinNumberComponent
Parts:
- removed D?: LED, LED_SMD:LED_0603_1608Metric_Pad1.05x0.95mm_HandSolder, symbol Device:LED_Small
- removed R?: 330, Resistor_SMD:R_0603_1608Metric_Pad0.98x0.95mm_HandSolder, symbol Device:R_Small
- JP1: renamed from JP?; footprint (none) -> Connector_PinHeader_2.00mm:PinHeader_1x03_P2.00mm_Vertical
Connections:
- net labels removed: LED4
- wire segments 352 -> 348
- no-connect marks 23 -> 24
Other:
- moved on the sheet: D1, D2, D3, R10, R8, R9

Commit message: uploadFloorplan
Parts:
- C5, C6: footprint Capacitor_SMD:C_0402_1005Metric -> Capacitor_SMD:C_0603_1608Metric
- U6: value PE4259 RF Switch -> SW409; footprint Package_TO_SOT_SMD:SOT-363_SC-70-6_Handsoldering -> CatSniffer:SW409; LCSC# (none) -> C391968; manf# (none) -> SW409; provedor (none) -> LCSC
- renumbered D3 to D1, D1 to D2, D2 to D3
Connections:
- no-connect marks 24 -> 23
Changed lines of the file:
@@
 P 20360 9390
 F 0 "U6" H 20360 9815 50  0000 C CNN
-F 1 "PE4259 RF Switch" H 20360 9724 50  0000 C CNN
-F 2 "Package_TO_SOT_SMD:SOT-363_SC-70-6_Handsoldering" H 20360 9490 50  0001 C CNN
-F 3 "http://cdn.macom.com/datasheets/maswss0115.pdf" H 20360 9490 50  0001 C CNN
+F 1 "SW409" H 20360 9724 50  0000 C CNN
+F 2 "CatSniffer:SW409" H 20360 9490 50  0001 C CNN
+F 3 "https://datasheet.lcsc.com/lcsc/1912111437_RFIC-SW409_C391968.pdf" H 20360 9490 50  0001 C CNN
+F 4 "C391968" H 20360 9390 50  0001 C CNN "LCSC#"
+F 5 "SW409" H 20360 9390 50  0001 C CNN "manf#"
+F 6 "LCSC" H 20360 9390 50  0001 C CNN "provedor"
 	1    20360 9390
 	1    0    0    -1
@@
 F 0 "C6" H 18945 8885 50  0000 L CNN
 F 1 "3.3pF" H 18870 8800 50  0000 L CNN
-F 2 "Capacitor_SMD:C_0402_1005Metric" H 19233 8670 50  0001 C CNN
+F 2 "Capacitor_SMD:C_0603_1608Metric" H 19233 8670 50  0001 C CNN
 F 3 "" H 19195 8820 50  0000 C CNN
 F 4 "GRM1885C1H3R3CA01D" H 19195 8820 50  0001 C CNN "manf#"
@@
 F 0 "C5" H 18445 8875 50  0000 L CNN
 F 1 "3.3pF" H 18370 8790 50  0000 L CNN
-F 2 "Capacitor_SMD:C_0402_1005Metric" H 18733 8660 50  0001 C CNN
+F 2 "Capacitor_SMD:C_0603_1608Metric" H 18733 8660 50  0001 C CNN
 F 3 "" H 18695 8810 50  0000 C CNN
 F 4 "GRM1885C1H3R3CA01D" H 18695 8810 50  0001 C CNN "manf#"
@@
 	5025 11850 5035 11850
 $Comp
-L Device:LED_Small D3
+L Device:LED_Small D1
 U 1 1 6087770B
 P 21500 6110
-F 0 "D3" V 21546 6040 50  0000 R CNN
+F 0 "D1" V 21546 6040 50  0000 R CNN
 F 1 "LED" V 21455 6040 50  0000 R CNN
 F 2 "LED_SMD:LED_0603_1608Metric_Pad1.05x0.95mm_HandSolder" V 21500 6110 50  0001 C CNN
@@
 	21500 5885 21500 6010
 $Comp
-L Device:LED_Small D1
+L Device:LED_Small D2
 U 1 1 6092AB5A
 P 21890 6100
-F 0 "D1" V 21936 6030 50  0000 R CNN
+F 0 "D2" V 21936 6030 50  0000 R CNN
 F 1 "LED" V 21845 6030 50  0000 R CNN
 F 2 "LED_SMD:LED_0603_1608Metric_Pad1.05x0.95mm_HandSolder" V 21890 6100 50  0001 C CNN
@@
 LED3
 $Comp
-L Device:LED_Small D2
+L Device:LED_Small D3
 U 1 1 6092B5D1
 P 22245 6100
-F 0 "D2" V 22291 6030 50  0000 R CNN
+F 0 "D3" V 22291 6030 50  0000 R CNN
 F 1 "LED" V 22200 6030 50  0000 R CNN
 F 2 "LED_SMD:LED_0603_1608Metric_Pad1.05x0.95mm_HandSolder" V 22245 6100 50  0001 C CNN
@@
 	1    0    0    -1
 $EndComp
-NoConn ~ 2290 2895
 $EndSCHEMATC

Commit message: fixSWDforSAMD21E
Parts:
- removed J5: Conn_01x04, Connector_PinHeader_1.00mm:PinHeader_1x04_P1.00mm_Vertical, symbol Connector_Generic:Conn_01x04
- added J1: Conn_01x06_Female, Connector:Tag-Connect_TC2030-IDC-NL_2x03_P1.27mm_Vertical, symbol Connector:Conn_01x06_Female
Connections:
- net labels added: RST
- wire segments 348 -> 351
- no-connect marks 23 -> 24
Changed lines of the file:
@@
 Wire Notes Line
 	5195 8215 11760 8215
-$Comp
-L Connector_Generic:Conn_01x04 J5
-U 1 1 5F63B8D3
-P 12710 6435
-F 0 "J5" H 12790 6427 50  0000 L CNN
-F 1 "Conn_01x04" H 12790 6336 50  0000 L CNN
-F 2 "Connector_PinHeader_1.00mm:PinHeader_1x04_P1.00mm_Vertical" H 12710 6435 50  0001 C CNN
-F 3 "~" H 12710 6435 50  0001 C CNN
-	1    12710 6435
-	1    0    0    -1
-$EndComp
-Wire Wire Line
-	12510 6335 12405 6335
-Wire Wire Line
-	12510 6435 12405 6435
-Wire Wire Line
-	12510 6535 12410 6535
-Wire Wire Line
-	12510 6635 12410 6635
-Text Label 12410 6535 2    50   ~ 0
+Text Label 12360 6340 2    50   ~ 0
 SWDIO
-Text Label 12405 6435 2    50   ~ 0
+Text Label 12360 6540 2    50   ~ 0
 SWCLK
 $Comp
 L power:GND #PWR040
 U 1 1 5F6EDB31
-P 12410 6635
-F 0 "#PWR040" H 12410 6385 50  0001 C CNN
-F 1 "GND" H 12415 6462 50  0000 C CNN
-F 2 "" H 12410 6635 50  0001 C CNN
-F 3 "" H 12410 6635 50  0001 C CNN
-	1    12410 6635
+P 12210 6705
+F 0 "#PWR040" H 12210 6455 50  0001 C CNN
+F 1 "GND" H 12215 6532 50  0000 C CNN
+F 2 "" H 12210 6705 50  0001 C CNN
+F 3 "" H 12210 6705 50  0001 C CNN
+	1    12210 6705
 	1    0    0    -1
 $EndComp
@@
 L power:+3V3 #PWR039
 U 1 1 5F6EEDB7
-P 12405 6335
-F 0 "#PWR039" H 12405 6185 50  0001 C CNN
-F 1 "+3V3" H 12420 6508 50  0000 C CNN
-F 2 "" H 12405 6335 50  0001 C CNN
-F 3 "" H 12405 6335 50  0001 C CNN
-	1    12405 6335
+P 12265 6155
+F 0 "#PWR039" H 12265 6005 50  0001 C CNN
+F 1 "+3V3" H 12280 6328 50  0000 C CNN
+F 2 "" H 12265 6155 50  0001 C CNN
+F 3 "" H 12265 6155 50  0001 C CNN
+	1    12265 6155
 	1    0    0    -1
 $EndComp
@@
 	1    0    0    -1
 $EndComp
+$Comp
+L Connector:Conn_01x06_Female J1
+U 1 1 60AB064F
+P 12640 6440
+F 0 "J1" H 12668 6416 50  0000 L CNN
+F 1 "Conn_01x06_Female" H 12668 6325 50  0000 L CNN
+F 2 "Connector:Tag-Connect_TC2030-IDC-NL_2x03_P1.27mm_Vertical" H 12640 6440 50  0001 C CNN
+F 3 "~" H 12640 6440 50  0001 C CNN
+	1    12640 6440
+	1    0    0    -1
+$EndComp
+Wire Wire Line
+	12440 6240 12265 6240
+Wire Wire Line
+	12265 6240 12265 6155
+Wire Wire Line
+	12440 6340 12360 6340
+Text Label 12355 6440 2    50   ~ 0
+RST
+Wire Wire Line
+	12440 6440 12355 6440
+Wire Wire Line
+	12440 6540 12360 6540
+Wire Wire Line
+	12440 6640 12210 6640
+Wire Wire Line
+	12210 6640 12210 6705
+NoConn ~ 12440 6740
 $EndSCHEMATC

Commit message: Modify schematic for better reading
Parts:
- added U?: ATSAMD21E18A, Package_QFP:TQFP-32_7x7mm_P0.8mm, symbol electroniccats:ATSAMD21E18A
- U3: symbol electroniccats:RFSW8006QTR7 -> CatStick-rescue:RFSW8006QTR7-electroniccats
- U8: MANUFACTURER Semtech -> (none); PARTREV 1.1 -> (none); STANDARD IPC-7351B -> (none)
Connections:
- net X48M_N: now reaches C7.1, U1.46 (X48M_N), Y2.3
- net X48M_P: now reaches C3.1, U1.47 (X48M_P), Y2.1
Other:
- note added: "JTAG - Matching CC1350 Launchpad"
- note added: "Main RF Switch"
- note added: "SAMD21 Main uC"
- note added: "Tx/Rx Switch"
- note removed: "ANTENNA"
- note removed: "JTAG - \nMatching CC1350 \nLaunchpad"
- note removed: "SWITCHING"
- moved on the sheet: BT1, C1, C10, C11, C12, C13, C14, C15, C16, C17, C18, C19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

Commit message: fixSAMDsch
Parts:
- removed C22, C23, C26: 0.1uF, Capacitor_SMD:C_0603_1608Metric, symbol Device:C_Small
- removed U7: ATSAMD21E18A-A, Package_QFP:TQFP-32_7x7mm_P0.8mm, symbol MCU_Microchip_SAMD:ATSAMD21E18A-A
- added C? (x3): 0.1uF, Capacitor_SMD:C_0603_1608Metric, symbol Device:C_Small
- added D?: LED, LED_SMD:LED_0603_1608Metric_Pad1.05x0.95mm_HandSolder, symbol Device:LED_Small
- added R?: 330, Resistor_SMD:R_0603_1608Metric_Pad0.98x0.95mm_HandSolder, symbol Device:R_Small
Connections:
- net +3V3: now also U?.30 (VDDIN), U?.9 (VDDA), C?.1, C?.2
- net ANT_SW: now also U?.27 (PA28/EINT8)
- net BUSY: now also U?.4 (PA03/EINT3/VREFA/AIN1)
- net CIPO: now also U?.21 (PA22/I2C/EINT6/SERCOM3+5.0)
- net COPI: now also U?.19 (PA18/EINT2/SERCOM1+3.2)
- net CTF1: now also U?.14 (PA11/EINT11/AIN19/SERCOM0+2.3/I2SF0)
- net CTF2: now also U?.16 (PA15/EINT15/SERCOM3+4.3)
- net CTF3: now also U?.17 (PA16/I2C/EINT0/SERCOM1+3.0)
- net CTS: now also U?.8 (PA07/EINT7/AIN7/SERCOM0.3/I2SD0)
- net D+: now also U?.24 (PA25/EINT13/SERCOM3+5.3/D+)
- net D-: now also U?.23 (PA24/EINT2/SERCOM3+5.2/D-)
- net DIO1: now also U?.1 (PA00/EINT0/SERCOM1.0)
- net DIO2: now also U?.2 (PA01/EINT1/SERCOM1.1)
- net DIO22: now also U?.25 (PA27/EINT15)
- net DIO3: now also U?.3 (PA02/EINT2/AIN0/Y0/VOUT)
- net GND: now also U?.10 (GND), U?.28 (GNDA), C?.1, C?.1, C?.2, R?.1
- net LED1: now also U?.11 (PA08/NMI/I2C/AIN16/SERCOM0+2.0/I2SD1)
- net LED2: now also U?.12 (PA09/I2C/EINT9/AIN17/SERCOM0+2.1/I2SMC)
- net LED3: now also U?.13 (PA10/EINT10/AIN18/SERCOM0+2.2/I2SCK), D?.2 (A); no longer D3.2 (A), U1.8 (DIO_3)
- net NSS: now also U?.18 (PA17/I2C/EINT1/SERCOM1+3.1)
- net RESET: now also U?.26 (/RESET)
- net RESET_CC: now also U?.15 (PA14/EINT14/SERCOM2+4.2)
- net RESET_SX: now also U?.22 (PA23/I2C/EINT7/SERCOM3+5.1/SOF)
- net RTS: now also U?.7 (PA06/EINT6/AIN6/SERCOM0.2)
- net RXD: now also U?.6 (PA05/EINT5/AIN5/SERCOM0.1)
- net SCK: now also U?.20 (PA19/EINT3/SERCOM1+3.3/I2SD0)
- net SWCLK: now also U?.31 (PA30/EINT10/SECOM1.2/SWCLK)
- net SWDIO: now also U?.32 (PA31/EINT11/SECOM1.3/SWDIO)
- net TXD: now also U?.5 (PA04/EINT4/VREFB/AIN4/SERCOM0.0)
- net at U?.29 (VDDCORE): now also C?.2
- new net: D?.1 (K), R?.2
- new net LED4: D3.2 (A), U1.8 (DIO_3)
Other:
- note removed: "SAMD21E"
- moved on the sheet: C28, D3, R8

Commit message: add line
Changed lines of the file:
@@
-	1    0    0    -1
-$EndComp
-$Comp
-L Connector:Conn_01x06_Female J1
-U 1 1 60AB064F
-P 17800 4990
-F 0 "J1" H 17828 4966 50  0000 L CNN
-F 1 "Conn_01x06_Female" H 17828 4875 50  0000 L CNN
-F 2 "Connector:Tag-Connect_TC2030-IDC-NL_2x03_P1.27mm_Vertical" H 17800 4990 50  0001 C CNN
-F 3 "~" H 17800 4990 50  0001 C CNN
-	1    17800 4990
 	1    0    0    -1
 $EndComp
@@
 Wire Notes Line
 	15685 5565 15685 10120
-Wire Notes Line
-	18955 5565 18955 10120
 Wire Wire Line
 	7415 1755 7415 1705
@@
 L power:+3V3 #PWR?
 U 1 1 610252E9
-P 12055 1475
-F 0 "#PWR?" H 12055 1325 50  0001 C CNN
-F 1 "+3V3" H 12070 1648 50  0000 C CNN
-F 2 "" H 12055 1475 50  0001 C CNN
-F 3 "" H 12055 1475 50  0001 C CNN
-	1    12055 1475
-	1    0    0    -1
-$EndComp
-Wire Wire Line
-	12055 1475 12055 1685
-Wire Wire Line
-	12055 1685 12160 1685
+P 12160 1425
+F 0 "#PWR?" H 12160 1275 50  0001 C CNN
+F 1 "+3V3" H 12175 1598 50  0000 C CNN
+F 2 "" H 12160 1425 50  0001 C CNN
+F 3 "" H 12160 1425 50  0001 C CNN
+	1    12160 1425
+	1    0    0    -1
+$EndComp
 Wire Wire Line
 	12660 4105 12255 4105
@@
 Wire Wire Line
 	12255 4105 12255 3905
+Wire Wire Line
+	12160 1425 12160 1555
+Wire Notes Line
+	18955 470  18955 10120
+$Comp
+L Connector:Conn_01x06_Female J1
+U 1 1 60AB064F
+P 17800 4990
+F 0 "J1" H 17828 4966 50  0000 L CNN
+F 1 "Conn_01x06_Female" H 17828 4875 50  0000 L CNN
+F 2 "Connector:Tag-Connect_TC2030-IDC-NL_2x03_P1.27mm_Vertical" H 17800 4990 50  0001 C CNN
+F 3 "~" H 17800 4990 50  0001 C CNN
+	1    17800 4990
+	1    0    0    -1
+$EndComp
 $EndSCHEMATC

Commit message: addResistorReset
Parts:
- added C41: 100nF, Capacitor_SMD:C_0603_1608Metric, symbol Device:C
- added R12: 100K, Resistor_SMD:R_0603_1608Metric_Pad0.98x0.95mm_HandSolder, symbol Device:R
- SW1, SW2: LCSC# C318889 -> C455281; manf# TS-1187A-C-C-B -> TS-1088R-02526
- gave numbers to parts that had none: 6
Connections:
- net GND: now also C41.2
- net RESET_CC: now also C41.1, R12.1
- net VDDS: now also R12.2
- net RESET_MCU: now reaches U1.21 (DIO_15)
- no-connect marks 24 -> 23
Changed lines of the file:
@@
 	1    0    0    -1
 $EndComp
-Text Label 3900 7335 0    60   ~ 0
+Text Label 4795 7260 0    60   ~ 0
 RESET_CC
 $Comp
@@
 Text Label 4350 5900 0    60   ~ 0
 SWITCH
-Text Label 1900 8135 2    60   ~ 0
-SWITCH
 $Comp
 L power:PWR_FLAG #FLG01
@@
 F 2 "Button_Switch_SMD:SW_SPST_TL3342" H 3650 6100 50  0001 C CNN
 F 3 "" H 3650 6100 50  0001 C CNN
-F 4 "C318889" H 3650 5900 50  0001 C CNN "LCSC#"
-F 5 "TS-1187A-C-C-B" H 3650 5900 50  0001 C CNN "manf#"
+F 4 "C455281" H 3650 5900 50  0001 C CNN "LCSC#"
+F 5 "TS-1088R-02526" H 3650 5900 50  0001 C CNN "manf#"
 F 6 "LCSC" H 3650 5900 50  0001 C CNN "provedor"
 	1    3650 5900
@@
 Wire Wire Line
 	7645 4355 7645 4455
-Wire Wire Line
-	3900 7335 3800 7335
 Connection ~ 1300 7735
 Wire Wire Line
 	1300 8235 1500 8235
-$Comp
-L Device:C C9
-U 1 1 5B9B4BB0
-P 3350 9235
-F 0 "C9" H 3465 9281 50  0000 L CNN
-F 1 "1uF" H 3465 9190 50  0000 L CNN
-F 2 "Capacitor_SMD:C_0603_1608Metric" H 3388 9085 50  0001 C CNN
-F 3 "~" H 3350 9235 50  0001 C CNN
-F 4 "0603F105M500NT" H 3350 9235 50  0001 C CNN "manf#"
-F 5 "LCSC" H 3350 9235 50  0001 C CNN "provedor"
-F 6 "C108343" H 3350 9235 50  0001 C CNN "LCSC#"
-	1    3350 9235
-	1    0    0    -1
-$EndComp
 $Comp
 L power:GND #PWR016
@@
 NoConn ~ 3250 6535
 NoConn ~ 3350 6535
-NoConn ~ 3150 9035
-Wire Wire Line
-	2000 8135 1900 8135
 $Comp
 L power:VCC #PWR036
@@
 F 2 "Button_Switch_SMD:SW_SPST_TL3342" H 17735 1305 50  0001 C CNN
 F 3 "~" H 17735 1305 50  0001 C CNN
-F 4 "C318889" H 17735 1105 50  0001 C CNN "LCSC#"
-F 5 "TS-1187A-C-C-B" H 17735 1105 50  0001 C CNN "manf#"
+F 4 "C455281" H 17735 1105 50  0001 C CNN "LCSC#"
+F 5 "TS-1088R-02526" H 17735 1105 50  0001 C CNN "manf#"
 F 6 "LCSC" H 17735 1105 50  0001 C CNN "provedor"
 	1    17735 1105
@@
 	21900 3615 22240 3615
 $Comp
-L electroniccats:ATSAMD21E18A U?
+L electroniccats:ATSAMD21E18A U7
 U 1 1 60DB2372
 P 13330 2765
-F 0 "U?" H 13695 4619 45  0000 C CNN
+F 0 "U7" H 13695 4619 45  0000 C CNN
 F 1 "ATSAMD21E18A" H 13695 4535 45  0000 C CNN
 F 2 "Package_QFP:TQFP-32_7x7mm_P0.8mm" H 13360 2915 20  0001 C CNN
@@
 $EndComp
 $Comp
-L power:GND #PWR?
+L power:GND #PWR0101
 U 1 1 61025FF6
 P 780 6775
-F 0 "#PWR?" H 780 6525 50  0001 C CNN
+F 0 "#PWR0101" H 780 6525 50  0001 C CNN
 F 1 "GND" H 780 6625 50  0000 C CNN
 F 2 "" H 780 6775 50  0000 C CNN
@@
 	780  6700 780  6775
 $Comp
-L power:GND #PWR?
+L power:GND #PWR0102
 U 1 1 61044B56
 P 1360 6765
-F 0 "#PWR?" H 1360 6515 50  0001 C CNN
+F 0 "#PWR0102" H 1360 6515 50  0001 C CNN
 F 1 "GND" H 1360 6615 50  0000 C CNN
 F 2 "" H 1360 6765 50  0000 C CNN
@@
 $EndComp
 $Comp
-L power:GND #PWR?
+L power:GND #PWR0103
 U 1 1 61110217
 P 1085 6770
-F 0 "#PWR?" H 1085 6520 50  0001 C CNN
+F 0 "#PWR0103" H 1085 6520 50  0001 C CNN
 F 1 "GND" H 1085 6620 50  0000 C CNN
 F 2 "" H 1085 6770 50  0000 C CNN
@@
 	14885 4165 14730 4165
 $Comp
-L Device:LED_Small D?
+L Device:LED_Small D4
 U 1 1 60C43107
 P 18045 2910
-F 0 "D?" V 18091 2840 50  0000 R CNN
+F 0 "D4" V 18091 2840 50  0000 R CNN
 F 1 "LED" V 18000 2840 50  0000 R CNN
 F 2 "LED_SMD:LED_0603_1608Metric_Pad1.05x0.95mm_HandSolder" V 18045 2910 50  0001 C CNN
@@
 $EndComp
 $Comp
-L Device:R_Small R?
+L Device:R_Small R11
 U 1 1 60C4376C
 P 18045 3225
-F 0 "R?" H 17925 3185 50  0000 C CNN
+F 0 "R11" H 17925 3185 50  0000 C CNN
 F 1 "330" H 17920 3265 50  0000 C CNN
 F 2 "Resistor_SMD:R_0603_1608Metric_Pad0.98x0.95mm_HandSolder" H 18045 3225 50  0001 C CNN
@@
 $EndComp
 $Comp
-L power:GND #PWR?
+L power:GND #PWR0104
 U 1 1 60C43D9A
 P 18045 3425
-F 0 "#PWR?" H 18045 3175 50  0001 C CNN
+F 0 "#PWR0104" H 18045 3175 50  0001 C CNN
 F 1 "GND" H 18050 3252 50  0000 C CNN
 F 2 "" H 18045 3425 50  0001 C CNN
@@
 	12540 1265 12660 1265
 $Comp
-L Device:C_Small C?
+L Device:C_Small C22
 U 1 1 60D6C661
 P 11935 1755
-F 0 "C?" V 11706 1755 50  0000 C CNN
+F 0 "C22" V 11706 1755 50  0000 C CNN
 F 1 "0.1uF" V 11797 1755 50  0000 C CNN
 F 2 "Capacitor_SMD:C_0603_1608Metric" H 11935 1755 50  0001 C CNN
@@
 	12255 3905 12660 3905
 $Comp
-L power:GND #PWR?
+L power:GND #PWR0105
 U 1 1 60E2B27F
 P 11935 1905
-F 0 "#PWR?" H 11935 1655 50  0001 C CNN
+F 0 "#PWR0105" H 11935 1655 50  0001 C CNN
 F 1 "GND" H 11940 1732 50  0000 C CNN
 F 2 "" H 11935 1905 50  0001 C CNN
@@
 	11935 1905 11935 1855
 $Comp
-L Device:C_Small C?
+L Device:C_Small C23
 U 1 1 60E51F71
 P 12160 1855
-F 0 "C?" H 12020 1780 50  0000 C CNN
+F 0 "C23" H 12020 1780 50  0000 C CNN
 F 1 "0.1uF" H 11985 1860 50  0000 C CNN
 F 2 "Capacitor_SMD:C_0603_1608Metric" H 12160 1855 50  0001 C CNN
@@
 	12160 1555 12660 1555
 $Comp
-L Device:C_Small C?
+L Device:C_Small C26
 U 1 1 60F84D56
 P 12525 1970
-F 0 "C?" H 12380 1920 50  0000 C CNN
+F 0 "C26" H 12380 1920 50  0000 C CNN
 F 1 "0.1uF" H 12345 1995 50  0000 C CNN
 F 2 "Capacitor_SMD:C_0603_1608Metric" H 12525 1970 50  0001 C CNN
@@
 	12525 1835 12525 1870
 $Comp
-L power:GND #PWR?
+L power:GND #PWR0106
 U 1 1 60FAE6B9
 P 12345 2180
-F 0 "#PWR?" H 12345 1930 50  0001 C CNN
+F 0 "#PWR0106" H 12345 1930 50  0001 C CNN
 F 1 "GND" H 12350 2007 50  0000 C CNN
 F 2 "" H 12345 2180 50  0001 C CNN
@@
 	12345 2105 12160 2105
 $Comp
-L power:+3V3 #PWR?
+L power:+3V3 #PWR0107
 U 1 1 610252E9
 P 12160 1425
-F 0 "#PWR?" H 12160 1275 50  0001 C CNN
+F 0 "#PWR0107" H 12160 1275 50  0001 C CNN
 F 1 "+3V3" H 12175 1598 50  0000 C CNN
 F 2 "" H 12160 1425 50  0001 C CNN
@@
 	1    0    0    -1
 $EndComp
+$Comp
+L Device:C C9
+U 1 1 5B9B4BB0
+P 3350 9235
+F 0 "C9" H 3465 9281 50  0000 L CNN
+F 1 "1uF" H 3465 9190 50  0000 L CNN
+F 2 "Capacitor_SMD:C_0603_1608Metric" H 3388 9085 50  0001 C CNN
+F 3 "~" H 3350 9235 50  0001 C CNN
+F 4 "0603F105M500NT" H 3350 9235 50  0001 C CNN "manf#"
+F 5 "LCSC" H 3350 9235 50  0001 C CNN "provedor"
+F 6 "C108343" H 3350 9235 50  0001 C CNN "LCSC#"
+	1    3350 9235
+	1    0    0    -1
+$EndComp
+$Comp
+L Device:C C41
+U 1 1 608CAAE2
+P 4575 7550
+F 0 "C41" H 4690 7596 50  0000 L CNN
+F 1 "100nF" H 4690 7505 50  0000 L CNN
+F 2 "Capacitor_SMD:C_0603_1608Metric" H 4613 7400 50  0001 C CNN
+F 3 "~" H 4575 7550 50  0001 C CNN
+F 4 "0603F105M500NT" H 4575 7550 50  0001 C CNN "manf#"
+F 5 "LCSC" H 4575 7550 50  0001 C CNN "provedor"
+F 6 "C108343" H 4575 7550 50  0001 C CNN "LCSC#"
+	1    4575 7550
+	1    0    0    -1
+$EndComp
+$Comp
+L Device:R R12
+U 1 1 608CB095
+P 4575 7145
+F 0 "R12" V 4655 7145 50  0000 C CNN
+F 1 "100K" V 4490 7145 50  0000 C CNN
+F 2 "Resistor_SMD:R_0603_1608Metric_Pad0.98x0.95mm_HandSolder" V 4505 7145 50  0001 C CNN
+F 3 "" H 4575 7145 50  0000 C CNN
+F 4 "C179820" H 4575 7145 50  0001 C CNN "LCSC#"
+F 5 "RT0603FRD07100KL" H 4575 7145 50  0001 C CNN "manf#"
+F 6 "LCSC" H 4575 7145 50  0001 C CNN "provedor"
+	1    4575 7145
+	-1   0    0    1
+$EndComp
+Wire Wire Line
+	2000 8135 1900 8135
+Text Label 1900 8135 2    60   ~ 0
+SWITCH
+Wire Wire Line
+	3150 9145 3150 9035
+Wire Wire Line
+	4575 7400 4575 7335
+$Comp
+L power:GND #PWR08
+U 1 1 6092EE43
+P 4575 7760
+F 0 "#PWR08" H 4575 7510 50  0001 C CNN
+F 1 "GND" H 4580 7587 50  0000 C CNN
+F 2 "" H 4575 7760 50  0001 C CNN
+F 3 "" H 4575 7760 50  0001 C CNN
+	1    4575 7760
+	1    0    0    -1
+$EndComp
+Wire Wire Line
+	4575 7760 4575 7700
+Text Label 4575 6875 0    50   ~ 0
+VDDS
+Wire Wire Line
+	4575 6995 4575 6875
+Wire Wire Line
+	3800 7335 4575 7335
+Connection ~ 4575 7335
+Wire Wire Line
+	4575 7335 4575 7295
+Wire Wire Line
+	4795 7260 4795 7335
+Wire Wire Line
+	4795 7335 4575 7335
+Text Label 3150 9145 3    50   ~ 0
+RESET_MCU
 $EndSCHEMATC
