File: hardware/CatStick.sch (KiCad schematic (older format))
At the start: 83 parts, among them J1 Conn_01x06_Female, J2 Antenna, J4 Conn_02x05_Odd_Even, P1 USB_C_Plug_USB2.0, Q1 DMN6140L, SW1 SW_Push, SW2 RST, U1 CC1352R1F3RGZR, U2 AP2112K-3.3, U3 RFSW8006QTR7, U4 0900FM15D0039, U5 0900PC15A0036, U6 SW409, U7 ATSAMD21E18A, U8 SX1262IMLTRT, Y1 32.768kHz, Y2 48MHz, Y3 32Mhz_10pF_10ppm

Commit message: addSAMDfootprint
Parts:
- SW1, SW2: footprint Button_Switch_SMD:SW_SPST_TL3342 -> Button_Switch_SMD:SW_SPST_EVQPE1
- U7: footprint Package_QFP:TQFP-32_7x7mm_P0.8mm -> Package_DFN_QFN:QFN-32-1EP_5x5mm_P0.5mm_EP3.65x3.65mm; Mouser# (none) -> ATSAMD21E18A-MUT; provedor (none) -> Mauser
Connections:
- net labels removed: RESET_CC, RESET_MCU
- wire segments 355 -> 353
- no-connect marks 23 -> 26
Changed lines of the file:
@@
 	1    0    0    -1
 $EndComp
-Text Label 4795 7260 0    60   ~ 0
-RESET_CC
 $Comp
 L Device:R R3
@@
 F 0 "SW1" H 3650 6185 50  0000 C CNN
 F 1 "SW_Push" H 3650 6094 50  0000 C CNN
-F 2 "Button_Switch_SMD:SW_SPST_TL3342" H 3650 6100 50  0001 C CNN
+F 2 "Button_Switch_SMD:SW_SPST_EVQPE1" H 3650 6100 50  0001 C CNN
 F 3 "" H 3650 6100 50  0001 C CNN
 F 4 "C455281" H 3650 5900 50  0001 C CNN "LCSC#"
@@
 Text Label 2950 9135 3    50   ~ 0
 TXD
-Text Label 3890 7935 0    50   ~ 0
-CTS
-Text Label 3890 8035 0    50   ~ 0
-RTS
-Wire Wire Line
-	3800 7935 3890 7935
-Wire Wire Line
-	3800 8035 3890 8035
 NoConn ~ 3800 7835
 $Comp
@@
 NoConn ~ 3050 9035
 NoConn ~ 2750 9035
-NoConn ~ 2000 8335
-NoConn ~ 2000 8235
 Text Label 17520 4890 2    50   ~ 0
 SWDIO
@@
 Text Label 14890 4365 0    50   ~ 0
 SWDIO
-Text Label 14880 4265 0    50   ~ 0
+Text Label 14885 4265 0    50   ~ 0
 SWCLK
 Text Label 14890 3165 0    50   ~ 0
@@
 F 0 "SW2" H 17735 1390 50  0000 C CNN
 F 1 "RST" H 17735 1299 50  0000 C CNN
-F 2 "Button_Switch_SMD:SW_SPST_TL3342" H 17735 1305 50  0001 C CNN
+F 2 "Button_Switch_SMD:SW_SPST_EVQPE1" H 17735 1305 50  0001 C CNN
 F 3 "~" H 17735 1305 50  0001 C CNN
 F 4 "C455281" H 17735 1105 50  0001 C CNN "LCSC#"
@@
 Text Label 14880 1865 0    50   ~ 0
 CTS
-Text Label 14890 2765 0    50   ~ 0
-RESET_CC
 Wire Wire Line
 	12370 7260 12285 7260
@@
 Wire Wire Line
 	21280 7890 21465 7890
-Text Label 1895 7935 2    50   ~ 0
-LED4
-Wire Wire Line
-	1895 7935 2000 7935
 Text Label 14885 4065 0    50   ~ 0
 DIO22
-$Comp
-L CatStick-rescue:CC1352R1F3RGZR-cc1352-cc1352-swim-thermo-rescue-CatStick-rescue U1
-U 1 1 5B86A9A7
-P 2850 7785
-F 0 "U1" H 2800 7735 50  0000 L CNN
-F 1 "CC1352R1F3RGZR" H 2500 7485 50  0000 L CNN
-F 2 "Package_DFN_QFN:VQFN-48-1EP_7x7mm_P0.5mm_EP5.15x5.15mm" H 3250 7035 50  0001 C CNN
-F 3 "" H 3250 7035 50  0001 C CNN
-F 4 " 595-CC1352P1F3RGZR" H 2850 7785 50  0001 C CNN "LCSC#"
-F 5 "595-CC1352R1F3RGZR " H 2850 7785 50  0001 C CNN "Mouser#"
-F 6 "CC1352R1F3RGZR " H 2850 7785 50  0001 C CNN "manf#"
-F 7 "Mouser" H 2850 7785 50  0001 C CNN "provedor"
-	1    2850 7785
-	1    0    0    -1
-$EndComp
 Wire Wire Line
 	17600 4790 17425 4790
@@
 F 0 "U7" H 13695 4619 45  0000 C CNN
 F 1 "ATSAMD21E18A" H 13695 4535 45  0000 C CNN
-F 2 "Package_QFP:TQFP-32_7x7mm_P0.8mm" H 13360 2915 20  0001 C CNN
+F 2 "Package_DFN_QFN:QFN-32-1EP_5x5mm_P0.5mm_EP3.65x3.65mm" H 13360 2915 20  0001 C CNN
 F 3 "https://www.mouser.mx/datasheet/2/268/SAM-D21-Family-Datasheet-DS40001882C-1381353.pdf" H 13330 2765 60  0001 C CNN
+F 4 "ATSAMD21E18A-MUT" H 13330 2765 50  0001 C CNN "Mouser#"
+F 5 "Mauser" H 13330 2765 50  0001 C CNN "provedor"
 	1    13330 2765
 	1    0    0    -1
@@
 Wire Wire Line
 	18045 2695 18045 2810
-Text Label 14890 2265 0    50   ~ 0
-LED3
 Wire Wire Line
 	14885 4265 14730 4265
@@
 	4795 7335 4575 7335
 Text Label 3150 9145 3    50   ~ 0
-RESET_MCU
+CTS
+NoConn ~ 3800 7935
+NoConn ~ 3800 8035
+$Comp
+L CatStick-rescue:CC1352R1F3RGZR-cc1352-cc1352-swim-thermo-rescue-CatStick-rescue U1
+U 1 1 5B86A9A7
+P 2850 7785
+F 0 "U1" H 2800 7735 50  0000 L CNN
+F 1 "CC1352R1F3RGZR" H 2500 7485 50  0000 L CNN
+F 2 "Package_DFN_QFN:VQFN-48-1EP_7x7mm_P0.5mm_EP5.15x5.15mm" H 3250 7035 50  0001 C CNN
+F 3 "" H 3250 7035 50  0001 C CNN
+F 4 " 595-CC1352P1F3RGZR" H 2850 7785 50  0001 C CNN "LCSC#"
+F 5 "595-CC1352R1F3RGZR " H 2850 7785 50  0001 C CNN "Mouser#"
+F 6 "CC1352R1F3RGZR " H 2850 7785 50  0001 C CNN "manf#"
+F 7 "Mouser" H 2850 7785 50  0001 C CNN "provedor"
+	1    2850 7785
+	1    0    0    -1
+$EndComp
+Text Label 1895 8335 2    50   ~ 0
+LED4
+NoConn ~ 2000 7935
+NoConn ~ 2000 8235
+Wire Wire Line
+	2000 8335 1895 8335
+Text Label 14890 2265 0    50   ~ 0
+LED3
+NoConn ~ 14890 2765
+Text Label 4795 7260 0    50   ~ 0
+RTS
 $EndSCHEMATC

Commit message: addButtonResetCC1352
Parts:
- removed C21: 100nF, Capacitor_SMD:C_0603_1608Metric, symbol Device:C
- removed R3: 100K, Resistor_SMD:R_0603_1608Metric_Pad0.98x0.95mm_HandSolder, symbol Device:R
- J4: footprint Connector_PinHeader_1.00mm:PinHeader_2x05_P1.00mm_Vertical -> Connector:Tag-Connect_TC2050-IDC-NL_2x05_P1.27mm_Vertical
Connections:
- net labels added: RESET_CC
- net labels removed: RESET_N, RST, SWITCH
- wire segments 353 -> 351
- no-connect marks 26 -> 27
Changed lines of the file:
@@
 $EndComp
-$Comp
-L Device:R R3
-U 1 1 58CA3762
-P 8885 8675
-F 0 "R3" V 8965 8675 50  0000 C CNN
-F 1 "100K" V 8885 8675 50  0000 C CNN
-F 2 "Resistor_SMD:R_0603_1608Metric_Pad0.98x0.95mm_HandSolder" V 8815 8675 50  0001 C CNN
-F 3 "" H 8885 8675 50  0000 C CNN
-F 4 "C179820" H 8885 8675 50  0001 C CNN "LCSC#"
-F 5 "RT0603FRD07100KL" H 8885 8675 50  0001 C CNN "manf#"
-F 6 "LCSC" H 8885 8675 50  0001 C CNN "provedor"
-	1    8885 8675
-	1    0    0    -1
-$EndComp
-$Comp
-L Device:C C21
-U 1 1 58CA3820
-P 8885 9275
-F 0 "C21" H 8910 9375 50  0000 L CNN
-F 1 "100nF" H 8910 9175 50  0000 L CNN
-F 2 "Capacitor_SMD:C_0603_1608Metric" H 8923 9125 50  0001 C CNN
-F 3 "" H 8885 9275 50  0000 C CNN
-F 4 "C14663" H 8885 9275 50  0001 C CNN "LCSC#"
-F 5 "LCSC" H 8885 9275 50  0001 C CNN "provedor"
-F 6 "CC0603KRX7R9BB104" H 8885 9275 50  0001 C CNN "manf#"
-	1    8885 9275
-	1    0    0    -1
-$EndComp
-$Comp
-L power:GND #PWR047
-U 1 1 58CA38E4
-P 8885 9525
-F 0 "#PWR047" H 8885 9275 50  0001 C CNN
-F 1 "GND" H 8885 9375 50  0000 C CNN
-F 2 "" H 8885 9525 50  0000 C CNN
-F 3 "" H 8885 9525 50  0000 C CNN
-	1    8885 9525
-	1    0    0    -1
-$EndComp
-Text Label 8735 9025 2    60   ~ 0
-RESET_N
 $Comp
 L power:GND #PWR035
@@
 	0    1    1    0
 $EndComp
-Text Label 4350 5900 0    60   ~ 0
-SWITCH
 $Comp
 L power:PWR_FLAG #FLG01
@@
 Connection ~ 7485 8875
 Wire Wire Line
-	8185 8875 8885 8875
-Wire Wire Line
 	8185 8775 8285 8775
 Wire Wire Line
@@
 	8185 8475 8285 8475
 Wire Wire Line
-	8885 8475 8885 8525
-Wire Wire Line
-	8885 8825 8885 8875
-Wire Wire Line
-	8885 9425 8885 9525
-Connection ~ 8885 8875
-Wire Wire Line
-	8735 9025 8885 9025
-Connection ~ 8885 9025
-Wire Wire Line
 	4035 1250 4035 1350
 Wire Wire Line
@@
 Wire Wire Line
 	7485 8875 7485 8975
-Wire Wire Line
-	8885 8875 8885 9025
-Wire Wire Line
-	8885 9025 8885 9125
 Wire Wire Line
 	5945 1705 6165 1705
@@
 F 0 "J4" H 7935 9092 50  0000 C CNN
 F 1 "Conn_02x05_Odd_Even" H 7935 9001 50  0000 C CNN
-F 2 "Connector_PinHeader_1.00mm:PinHeader_2x05_P1.00mm_Vertical" H 7885 8675 50  0001 C CNN
+F 2 "Connector:Tag-Connect_TC2050-IDC-NL_2x05_P1.27mm_Vertical" H 7885 8675 50  0001 C CNN
 F 3 "~" H 7885 8675 50  0001 C CNN
 	1    7885 8675
@@
 Wire Wire Line
 	7385 8475 7685 8475
-$Comp
-L power:VCC #PWR046
-U 1 1 5B9CE581
-P 8885 8475
-F 0 "#PWR046" H 8885 8325 50  0001 C CNN
-F 1 "VCC" H 8902 8648 50  0000 C CNN
-F 2 "" H 8885 8475 50  0001 C CNN
-F 3 "" H 8885 8475 50  0001 C CNN
-	1    8885 8475
-	1    0    0    -1
-$EndComp
 Text Notes 485  5225 0    89   ~ 0
 CC1352
@@
 Text Label 14885 3765 0    50   ~ 0
 RESET_SX
-Text Label 14880 1765 0    50   ~ 0
-RTS
 Text Label 14880 1865 0    50   ~ 0
 CTS
@@
 Wire Wire Line
 	17600 4890 17520 4890
-Text Label 17515 4990 2    50   ~ 0
-RST
 Wire Wire Line
 	17600 4990 17515 4990
@@
 $EndComp
 Wire Wire Line
-	2000 8135 1900 8135
-Text Label 1900 8135 2    60   ~ 0
-SWITCH
-Wire Wire Line
-	3150 9145 3150 9035
+	3150 9355 3150 9095
 Wire Wire Line
 	4575 7400 4575 7335
@@
 	4575 7335 4575 7295
 Wire Wire Line
-	4795 7260 4795 7335
-Wire Wire Line
 	4795 7335 4575 7335
-Text Label 3150 9145 3    50   ~ 0
+Text Label 3150 9355 3    50   ~ 0
 CTS
 NoConn ~ 3800 7935
@@
 LED3
 NoConn ~ 14890 2765
-Text Label 4795 7260 0    50   ~ 0
+Text Label 4795 7155 0    50   ~ 0
+RESET_CC
+Text Label 17515 4990 2    50   ~ 0
+RESET
+Text Label 14880 1765 0    50   ~ 0
 RTS
+Text Label 5035 7340 0    50   ~ 0
+RTS
+Wire Wire Line
+	5035 7340 4795 7340
+Wire Wire Line
+	4795 7155 4795 7335
+Connection ~ 4795 7335
+Wire Wire Line
+	4795 7335 4795 7340
+Text Label 8295 8875 0    50   ~ 0
+RESET_CC
+Wire Wire Line
+	8295 8875 8185 8875
+Wire Wire Line
+	3150 9095 3005 9095
+Wire Wire Line
+	3005 9095 3005 9350
+Connection ~ 3150 9095
+Wire Wire Line
+	3150 9095 3150 9035
+NoConn ~ 2000 8135
+Text Label 4350 5900 0    50   ~ 0
+RESET_CC
+Text Label 3005 9350 3    50   ~ 0
+RESET_CC
 $EndSCHEMATC

Commit message: FloorplanInProgress
Parts:
- SW1, SW2: footprint Button_Switch_SMD:SW_SPST_EVQPE1 -> CatSniffer:TS1088R02026
Changed lines of the file:
@@
 F 0 "SW1" H 3650 6185 50  0000 C CNN
 F 1 "SW_Push" H 3650 6094 50  0000 C CNN
-F 2 "Button_Switch_SMD:SW_SPST_EVQPE1" H 3650 6100 50  0001 C CNN
+F 2 "CatSniffer:TS1088R02026" H 3650 6100 50  0001 C CNN
 F 3 "" H 3650 6100 50  0001 C CNN
 F 4 "C455281" H 3650 5900 50  0001 C CNN "LCSC#"
@@
 F 0 "SW2" H 17735 1390 50  0000 C CNN
 F 1 "RST" H 17735 1299 50  0000 C CNN
-F 2 "Button_Switch_SMD:SW_SPST_EVQPE1" H 17735 1305 50  0001 C CNN
+F 2 "CatSniffer:TS1088R02026" H 17735 1305 50  0001 C CNN
 F 3 "~" H 17735 1305 50  0001 C CNN
 F 4 "C455281" H 17735 1105 50  0001 C CNN "LCSC#"

Commit message: BatteryRemove
Parts:
- removed BT1: a, Connector_Molex:Molex_KK-254_AE-6410-02A_1x02_P2.54mm_Vertical, symbol Device:Battery
- removed Q1: DMN6140L, Package_TO_SOT_SMD:SOT-23, symbol Transistor_FET:DMN6140L
- removed R1: 10K, Resistor_SMD:R_0603_1608Metric_Pad0.98x0.95mm_HandSolder, symbol Device:R_Small
- removed R2: 100K, Resistor_SMD:R_0603_1608Metric_Pad0.98x0.95mm_HandSolder, symbol Device:R
- added BOOT1: SW_Push, CatSniffer:TS1088R02026, symbol Switch:SW_Push
- JP1: footprint Connector_PinHeader_2.00mm:PinHeader_1x03_P2.00mm_Vertical -> Jumper:SolderJumper-3_P1.3mm_Bridged12_RoundedPad1.0x1.5mm_NumberLabels
- renumbered SW2 to RESET1, SW1 to RESET_CC1
Connections:
- net labels added: BOOT
- net labels removed: +BATT
- wire segments 351 -> 344
Other:
- moved on the sheet: C10, C8, RESET_CC1, U2

Commit message: fix source for cc1352
Parts:
- removed C28: 0.1uF, Capacitor_SMD:C_0603_1608Metric, symbol Device:C_Small
- J4: value Conn_02x05_Odd_Even -> JTAG
- U7: symbol electroniccats:ATSAMD21E18A -> CatStick-rescue:ATSAMD21E18A-electroniccats
Connections:
- net +3V3: now also J4.1 (Pin_1), L3.2
- net VCC: no longer J4.1 (Pin_1), L3.2
Other:
- note added: "JTAG - Matching CC1350"
- note added: "LEDS"
- note added: "MAIN RF SWITCH"
- note added: "MICROCONTROLLER"
- note added: "SWD FOR SAMD21"
- note added: "SWITCH LORA"
- note removed: "1.8-3.8 V"
- note removed: "JTAG - Matching CC1350 Launchpad"
- note removed: "LEDs\n\n\n"
- note removed: "Main RF Switch"
- note removed: "SAMD21 Main uC"
- note removed: "SWD FOR SAMD21E"
- note removed: "Tx/Rx Switch"
- moved on the sheet: BOOT1, C10, C22, C23, C26, C35, C36, C38, C39, C8, D1, D2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

Commit message: fixCrossSignals
Parts:
- added C21, C28: 47pF, Capacitor_SMD:C_0603_1608Metric, symbol Device:C
Connections:
- net SW_RFI: now also C28.1; no longer U6.1 (RF1)
- net SW_RFO: now also C21.1; no longer U6.3 (RF2)
- net UBP_2_4_GHZ: now also C36.1; no longer C38.1
- net UBP_SUB-1_GHZ: now also C38.1; no longer C36.1
- new net: C21.2, U6.1 (RF1)
- new net: C28.2, U6.3 (RF2)
Changed lines of the file:
@@
 Text Label 20425 3460 2    50   ~ 0
 CTF3
+Text Label 19760 2785 2    50   ~ 0
+UBP_2_4_GHZ
 Text Label 19630 3050 2    50   ~ 0
-UBP_2_4_GHZ
-Text Label 19760 2785 2    50   ~ 0
 UBP_SUB-1_GHZ
 $Comp
@@
 	20470 7235 20570 7235
 Wire Wire Line
-	19670 7135 19555 7135
-Wire Wire Line
-	19670 7335 19565 7335
-Wire Wire Line
 	19970 7735 19970 7795
 $Comp
@@
 	-1   0    0    -1
 $EndComp
-Text Label 19565 7335 2    50   ~ 0
+Text Label 19150 7135 2    50   ~ 0
 SW_RFO
-Text Label 19555 7135 2    50   ~ 0
+Text Label 19160 7335 2    50   ~ 0
 SW_RFI
 Text Label 14670 4205 0    50   ~ 0
@@
 	11945 1865 11945 1995
 Wire Notes Line
-	18955 470  18955 10120
+	18840 480  18840 10130
 $Comp
 L Connector:Conn_01x06_Female J1
@@
 LEDS
 $Comp
-L power:+3V3 #PWR?
+L power:+3V3 #PWR01
 U 1 1 60C1A6B6
 P 1450 4015
-F 0 "#PWR?" H 1450 3865 50  0001 C CNN
+F 0 "#PWR01" H 1450 3865 50  0001 C CNN
 F 1 "+3V3" H 1465 4188 50  0000 C CNN
 F 2 "" H 1450 4015 50  0001 C CNN
@@
 $EndComp
 $Comp
-L power:+3V3 #PWR?
+L power:+3V3 #PWR02
 U 1 1 60C1D5F0
 P 7385 8475
-F 0 "#PWR?" H 7385 8325 50  0001 C CNN
+F 0 "#PWR02" H 7385 8325 50  0001 C CNN
 F 1 "+3V3" H 7400 8648 50  0000 C CNN
 F 2 "" H 7385 8475 50  0001 C CNN
@@
 	1    0    0    -1
 $EndComp
+$Comp
+L Device:C C21
+U 1 1 60977A2F
+P 19360 7135
+F 0 "C21" V 19505 6965 50  0000 L CNN
+F 1 "47pF" V 19420 6910 50  0000 L CNN
+F 2 "Capacitor_SMD:C_0603_1608Metric" H 19398 6985 50  0001 C CNN
+F 3 "" H 19360 7135 50  0000 C CNN
+F 4 "LCSC" H 19360 7135 50  0001 C CNN "provedor"
+F 5 "C14858" H 19360 7135 50  0001 C CNN "LCSC#"
+F 6 "CL10C101JB8NNNC" H 19360 7135 50  0001 C CNN "manf#"
+	1    19360 7135
+	0    -1   -1   0
+$EndComp
+$Comp
+L Device:C C28
+U 1 1 60977E80
+P 19370 7335
+F 0 "C28" V 19325 7125 50  0000 L CNN
+F 1 "47pF" V 19250 7100 50  0000 L CNN
+F 2 "Capacitor_SMD:C_0603_1608Metric" H 19408 7185 50  0001 C CNN
+F 3 "" H 19370 7335 50  0000 C CNN
+F 4 "LCSC" H 19370 7335 50  0001 C CNN "provedor"
+F 5 "C14858" H 19370 7335 50  0001 C CNN "LCSC#"
+F 6 "CL10C101JB8NNNC" H 19370 7335 50  0001 C CNN "manf#"
+	1    19370 7335
+	0    -1   -1   0
+$EndComp
+Wire Wire Line
+	19520 7335 19670 7335
+Wire Wire Line
+	19160 7335 19220 7335
+Wire Wire Line
+	19510 7135 19670 7135
+Wire Wire Line
+	19150 7135 19210 7135
 $EndSCHEMATC

Commit message: addUserSwitch
Parts:
- added SW1: SW1, CatSniffer:TS1088R02026, symbol Switch:SW_Push
- BOOT1: value SW_Push -> BOOT
- J4: manf# (none) -> TC2050-IDC-ND; provedor (none) -> Digikey
- RESET1: value RST -> RESET
- RESET_CC1: value SW_Push -> RESET_CC
Connections:
- net GND: now also SW1.2
- net U_SWITCH: now reaches U7.15 (PA14/EINT14/SERCOM2+4.2)
- net U_SWITCH: now also SW1.1
- no-connect marks 27 -> 26
Other:
- moved on the sheet: BOOT1, RESET1, RESET_CC1
Changed lines of the file:
@@
 L power:GND #PWR035
 U 1 1 58CC4391
-P 8565 1475
-F 0 "#PWR035" H 8565 1225 50  0001 C CNN
-F 1 "GND" H 8565 1325 50  0000 C CNN
-F 2 "" H 8565 1475 50  0000 C CNN
-F 3 "" H 8565 1475 50  0000 C CNN
-	1    8565 1475
+P 7830 1290
+F 0 "#PWR035" H 7830 1040 50  0001 C CNN
+F 1 "GND" H 7830 1140 50  0000 C CNN
+F 2 "" H 7830 1290 50  0000 C CNN
+F 3 "" H 7830 1290 50  0000 C CNN
+	1    7830 1290
 	1    0    0    -1
 $EndComp
@@
 	8185 8475 8285 8475
 Wire Wire Line
-	8565 1475 8665 1475
-Wire Wire Line
-	9065 1475 9165 1475
+	7830 1290 7930 1290
+Wire Wire Line
+	8330 1290 8430 1290
 Wire Wire Line
 	1300 8235 1200 8235
@@
 F 2 "Connector:Tag-Connect_TC2050-IDC-NL_2x05_P1.27mm_Vertical" H 7885 8675 50  0001 C CNN
 F 3 "~" H 7885 8675 50  0001 C CNN
+F 4 "TC2050-IDC-ND" H 7885 8675 50  0001 C CNN "manf#"
+F 5 "Digikey" H 7885 8675 50  0001 C CNN "provedor"
 	1    7885 8675
 	1    0    0    -1
@@
 L Switch:SW_Push RESET_CC1
 U 1 1 5BAA6E6C
-P 8865 1475
-F 0 "RESET_CC1" H 8865 1760 50  0000 C CNN
-F 1 "SW_Push" H 8865 1669 50  0000 C CNN
-F 2 "CatSniffer:TS1088R02026" H 8865 1675 50  0001 C CNN
-F 3 "" H 8865 1675 50  0001 C CNN
-F 4 "C455281" H 8865 1475 50  0001 C CNN "LCSC#"
-F 5 "TS-1088R-02526" H 8865 1475 50  0001 C CNN "manf#"
-F 6 "LCSC" H 8865 1475 50  0001 C CNN "provedor"
-	1    8865 1475
+P 8130 1290
+F 0 "RESET_CC1" H 8130 1575 50  0000 C CNN
+F 1 "RESET_CC" H 8130 1484 50  0000 C CNN
+F 2 "CatSniffer:TS1088R02026" H 8130 1490 50  0001 C CNN
+F 3 "" H 8130 1490 50  0001 C CNN
+F 4 "C455281" H 8130 1290 50  0001 C CNN "LCSC#"
+F 5 "TS-1088R-02526" H 8130 1290 50  0001 C CNN "manf#"
+F 6 "LCSC" H 8130 1290 50  0001 C CNN "provedor"
+	1    8130 1290
 	1    0    0    -1
 $EndComp
@@
 L Switch:SW_Push RESET1
 U 1 1 5FD003C3
-P 9050 2910
-F 0 "RESET1" H 9050 3195 50  0000 C CNN
-F 1 "RST" H 9050 3104 50  0000 C CNN
-F 2 "CatSniffer:TS1088R02026" H 9050 3110 50  0001 C CNN
-F 3 "~" H 9050 3110 50  0001 C CNN
-F 4 "C455281" H 9050 2910 50  0001 C CNN "LCSC#"
-F 5 "TS-1088R-02526" H 9050 2910 50  0001 C CNN "manf#"
-F 6 "LCSC" H 9050 2910 50  0001 C CNN "provedor"
-	1    9050 2910
-	1    0    0    -1
-$EndComp
-Text Label 8700 2910 2    50   ~ 0
+P 9750 2005
+F 0 "RESET1" H 9750 2290 50  0000 C CNN
+F 1 "RESET" H 9750 2199 50  0000 C CNN
+F 2 "CatSniffer:TS1088R02026" H 9750 2205 50  0001 C CNN
+F 3 "~" H 9750 2205 50  0001 C CNN
+F 4 "C455281" H 9750 2005 50  0001 C CNN "LCSC#"
+F 5 "TS-1088R-02526" H 9750 2005 50  0001 C CNN "manf#"
+F 6 "LCSC" H 9750 2005 50  0001 C CNN "provedor"
+	1    9750 2005
+	1    0    0    -1
+$EndComp
+Text Label 9400 2005 2    50   ~ 0
 RESET
 Wire Wire Line
-	8700 2910 8850 2910
+	9400 2005 9550 2005
 $Comp
 L power:GND #PWR042
 U 1 1 5FD0172F
-P 9355 2965
-F 0 "#PWR042" H 9355 2715 50  0001 C CNN
-F 1 "GND" H 9360 2792 50  0000 C CNN
-F 2 "" H 9355 2965 50  0001 C CNN
-F 3 "" H 9355 2965 50  0001 C CNN
-	1    9355 2965
-	1    0    0    -1
-$EndComp
-Wire Wire Line
-	9355 2910 9355 2965
-Wire Wire Line
-	9250 2910 9355 2910
+P 10055 2060
+F 0 "#PWR042" H 10055 1810 50  0001 C CNN
+F 1 "GND" H 10060 1887 50  0000 C CNN
+F 2 "" H 10055 2060 50  0001 C CNN
+F 3 "" H 10055 2060 50  0001 C CNN
+	1    10055 2060
+	1    0    0    -1
+$EndComp
+Wire Wire Line
+	10055 2005 10055 2060
+Wire Wire Line
+	9950 2005 10055 2005
 $Comp
 L SX1262IMLTRT:SX1262IMLTRT U8
@@
 Text Label 14675 2705 0    50   ~ 0
 LED3
-NoConn ~ 14675 3205
 Text Label 4795 7155 0    50   ~ 0
 RESET_CC
@@
 	8295 8875 8185 8875
 NoConn ~ 2000 8135
-Text Label 9165 1475 0    50   ~ 0
+Text Label 8430 1290 0    50   ~ 0
 RESET_CC
 Text Label 3005 9350 3    50   ~ 0
@@
 L Switch:SW_Push BOOT1
 U 1 1 60C2B98F
-P 8920 2150
-F 0 "BOOT1" H 8920 2435 50  0000 C CNN
-F 1 "SW_Push" H 8920 2344 50  0000 C CNN
-F 2 "CatSniffer:TS1088R02026" H 8920 2350 50  0001 C CNN
-F 3 "" H 8920 2350 50  0001 C CNN
-F 4 "C455281" H 8920 2150 50  0001 C CNN "LCSC#"
-F 5 "TS-1088R-02526" H 8920 2150 50  0001 C CNN "manf#"
-F 6 "LCSC" H 8920 2150 50  0001 C CNN "provedor"
-	1    8920 2150
+P 8185 1965
+F 0 "BOOT1" H 8185 2250 50  0000 C CNN
+F 1 "BOOT" H 8185 2159 50  0000 C CNN
+F 2 "CatSniffer:TS1088R02026" H 8185 2165 50  0001 C CNN
+F 3 "" H 8185 2165 50  0001 C CNN
+F 4 "C455281" H 8185 1965 50  0001 C CNN "LCSC#"
+F 5 "TS-1088R-02526" H 8185 1965 50  0001 C CNN "manf#"
+F 6 "LCSC" H 8185 1965 50  0001 C CNN "provedor"
+	1    8185 1965
 	1    0    0    -1
 $EndComp
@@
 L power:GND #PWR0108
 U 1 1 60C4D0C5
-P 8625 2230
-F 0 "#PWR0108" H 8625 1980 50  0001 C CNN
-F 1 "GND" H 8625 2080 50  0000 C CNN
-F 2 "" H 8625 2230 50  0000 C CNN
-F 3 "" H 8625 2230 50  0000 C CNN
-	1    8625 2230
-	1    0    0    -1
-$EndComp
-Wire Wire Line
-	8625 2230 8625 2150
-Wire Wire Line
-	8625 2150 8720 2150
-Wire Wire Line
-	9180 2150 9120 2150
-Text Label 9180 2150 0    50   ~ 0
+P 7890 2045
+F 0 "#PWR0108" H 7890 1795 50  0001 C CNN
+F 1 "GND" H 7890 1895 50  0000 C CNN
+F 2 "" H 7890 2045 50  0000 C CNN
+F 3 "" H 7890 2045 50  0000 C CNN
+	1    7890 2045
+	1    0    0    -1
+$EndComp
+Wire Wire Line
+	7890 2045 7890 1965
+Wire Wire Line
+	7890 1965 7985 1965
+Wire Wire Line
+	8445 1965 8385 1965
+Text Label 8445 1965 0    50   ~ 0
 BOOT
 Wire Notes Line
@@
 Wire Wire Line
 	19150 7135 19210 7135
+$Comp
+L Switch:SW_Push SW1
+U 1 1 60AC93F3
+P 9925 1285
+F 0 "SW1" H 9925 1570 50  0000 C CNN
+F 1 "SW1" H 9925 1479 50  0000 C CNN
+F 2 "CatSniffer:TS1088R02026" H 9925 1485 50  0001 C CNN
+F 3 "" H 9925 1485 50  0001 C CNN
+F 4 "C455281" H 9925 1285 50  0001 C CNN "LCSC#"
+F 5 "TS-1088R-02526" H 9925 1285 50  0001 C CNN "manf#"
+F 6 "LCSC" H 9925 1285 50  0001 C CNN "provedor"
+	1    9925 1285
+	1    0    0    -1
+$EndComp
+Text Label 9515 1285 2    50   ~ 0
+U_SWITCH
+$Comp
+L power:GND #PWR06
+U 1 1 60AC9DB0
+P 10155 1445
+F 0 "#PWR06" H 10155 1195 50  0001 C CNN
+F 1 "GND" H 10155 1295 50  0000 C CNN
+F 2 "" H 10155 1445 50  0000 C CNN
+F 3 "" H 10155 1445 50  0000 C CNN
+	1    10155 1445
+	1    0    0    -1
+$EndComp
+Wire Wire Line
+	9515 1285 9725 1285
+Wire Wire Line
+	10155 1445 10155 1285
+Wire Wire Line
+	10155 1285 10125 1285
+Text Label 14675 3205 0    50   ~ 0
+U_SWITCH
 $EndSCHEMATC

Commit message: updateBoom
Parts:
- BOOT1: value BOOT -> SW
- C30: renamed from C21; LCSC# C14858 -> C519486; manf# CL10C101JB8NNNC -> CC0603FRNPO9BN470
- C32: renamed from C28; LCSC# C14858 -> C519486; manf# CL10C101JB8NNNC -> CC0603FRNPO9BN470
- J1: renamed from J2; LCSC# (none) -> C1509219; manf# (none) -> HJ-SMA023; provedor (none) -> LCSC
- RESET1: value RESET -> SW
- RESET_CC1: value RESET_CC -> SW
- SW1: value SW1 -> SW
- renumbered C8 to C1, C18 to C10, C19 to C11, C20 to C12, C11 to C13, C12 to C14, C13 to C15, C14 to C16, C15 to C17, C16 to C18, C17 to C19, C10 to C2, C3 to C20, C7 to C21, C4 to C22, C31 to C23, C32 to C24, C37 to C25, C29 to C26, C5 to C27, C6 to C28, C40 to C29, C22 to C3, C24 to C31, C41 to C34, C30 to C35, C1 to C36, C34 to C37, C2 to C38, C25 to C39, C23 to C4, C27 to C40, C9 to C41, C26 to C5, C35 to C6, C36 to C7, C38 to C8, C39 to C9, D4 to D1, D1 to D3, D3 to D4, J1 to J2, J4 to J3, L3 to L1, L4 to L2, L1 to L3, L7 to L4, L6 to L5, R6 to R1, R7 to R2, R11 to R3, R9 to R4, R10 to R5, R12 to R6, R4 to R7, R5 to R8, R8 to R9, U2 to U1, U3 to U2, U7 to U3, U5 to U4, U4 to U5, U8 to U7, U1 to U8, Y2 to Y1, Y1 to Y2
Other:
- note removed: "I2C:"
