File: hardware/CatStick.kicad_pcb (KiCad board)
At the start: 4 copper layers, 80 x 20 mm, 82 parts, among them J1 Conn_01x06_Female, J2 Antenna, J4 JTAG, P1 USB_C_Plug_USB2.0, U1 CC1352R1F3RGZR, U2 AP2112K-3.3, U3 RFSW8006QTR7, U4 0900FM15D0039, U5 0900PC15A0036, U6 SW409, U7 ATSAMD21E18A, U8 SX1262IMLTRT, Y1 32.768kHz, Y2 48MHz, Y3 32Mhz_10pF_10ppm

Commit message: fixCrossSignals
Parts:
- added C21: 47pF, Capacitor_SMD:C_0603_1608Metric, F.Cu at (142.8, 103.9)
- added C28: 47pF, Capacitor_SMD:C_0603_1608Metric, F.Cu at (142.8, 105.7)
- moved R12 35.6 mm to (132.8, 93.9), turned to 90 degrees
- moved L4 28.7 mm to (111.8, 94.1), turned to 270 degrees
- moved C9 26.4 mm to (132.8, 109.7)
- moved C18 25.5 mm to (113.4, 94.3), turned to 270 degrees
- moved C19 22.4 mm to (115.0, 94.3), turned to 270 degrees
- moved C41 19.6 mm to (132.0, 117.1), turned to 180 degrees
- moved C20 19.2 mm to (116.6, 94.3), turned to 270 degrees
- moved C17 16.0 mm to (118.2, 94.3), turned to 270 degrees
- moved C16 12.9 mm to (119.8, 94.3), turned to 270 degrees
- moved C15 9.67 mm to (121.4, 94.3), turned to 270 degrees
- moved L3 6.53 mm to (129.3, 94.1), turned to 270 degrees
- moved C14 6.40 mm to (123.0, 94.3), turned to 270 degrees
- moved C38 3.83 mm to (149.5, 114.0)
- moved C11 3.43 mm to (127.8, 94.3), turned to 270 degrees
- moved C13 3.31 mm to (124.6, 94.3), turned to 270 degrees
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Connections:
- C36 pad 1: /UBP_SUB-1_GHZ -> /UBP_2_4_GHZ
- C38 pad 1: /UBP_2_4_GHZ -> /UBP_SUB-1_GHZ
- U6 pad 1: /SW_RFI -> Net-(C21-Pad2)
- U6 pad 3: /SW_RFO -> Net-(C28-Pad2)

Commit message: addUserSwitch
Parts:
- added SW1: SW1, CatSniffer:TS1088R02026, F.Cu at (112.5, 102.7)
- BOOT: renamed from BOOT1; value SW_Push -> BOOT
- RESET: renamed from RESET1; value RST -> RESET
- RESET_CC: renamed from RESET_CC1; value SW_Push -> RESET_CC
- moved C30 28.5 mm to (126.8, 110.4)
- moved L6 27.9 mm to (125.6, 111.4)
- moved J1 21.4 mm to (154.4, 102.2)
- moved R12 16.2 mm to (116.6, 94.1), turned to 270 degrees
- moved C31 15.3 mm to (146.0, 84.2)
- moved L7 15.3 mm to (147.1, 85.2)
- moved C29 15.3 mm to (143.5, 84.8)
- moved C27 15.3 mm to (138.1, 88.8)
- moved C24 15.3 mm to (142.4, 85.9)
- moved C25 15.3 mm to (138.4, 85.3)
- moved C32 15.3 mm to (144.9, 83.1)
- moved Y3 15.3 mm to (139.9, 87.1)
- moved BOOT 7.07 mm to (128.1, 102.7)
- moved RESET_CC 6.95 mm to (120.2, 102.7)
- moved J4 5.46 mm to (120.5, 129.7)
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Connections:
- U7 pad 15: Net-(U7-Pad15) -> /U_SWITCH

Commit message: floorPlan
Parts:
- removed SW1: SW1, CatSniffer:TS1088R02026
- added SW: SW1, CatSniffer:TS1088R02026, F.Cu at (119.6, 102.7)
- moved J1 50.0 mm to (104.4, 102.3)
- moved L4 26.7 mm to (129.8, 111.2)
- moved C24 26.0 mm to (132.8, 110.1), turned to 180 degrees
- moved C29 25.9 mm to (132.8, 108.5), turned to 180 degrees
- moved C18 24.3 mm to (128.2, 111.3), turned to 90 degrees
- moved D3 23.5 mm to (99.3, 119.0)
- moved R8 23.5 mm to (95.8, 119.0)
- moved C19 22.2 mm to (126.7, 111.3), turned to 90 degrees
- moved C41 21.7 mm to (113.2, 112.5)
- moved C20 20.3 mm to (125.1, 111.3), turned to 90 degrees
- moved BOOT 19.6 mm to (114.9, 117.2)
- moved RESET_CC 19.5 mm to (107.2, 117.2)
- moved L7 19.4 mm to (139.8, 103.2), turned to 0 degrees
- moved C32 19.1 mm to (140.0, 101.6), turned to 180 degrees
- moved C31 18.0 mm to (142.3, 101.8), turned to 270 degrees
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
Commit message: updateBoom
Parts:
- BOOT: value BOOT -> SW
- RESET: value RESET -> SW
- RESET_CC: value RESET_CC -> SW
- SW: value SW1 -> SW
- moved C25 1.41 mm to (151.5, 116.5)
- moved C7 1.11 mm to (155.3, 117.3)
- moved C8 0.76 mm to (154.0, 113.8), turned to 90 degrees
- moved J1 0.47 mm to (165.0, 110.1)
- renumbered C8 to C1, C18 to C10, C19 to C11, C20 to C12, C11 to C13, C12 to C14, C13 to C15, C14 to C16, C15 to C17, C16 to C18, C17 to C19, C10 to C2, C3 to C20, C7 to C21, C4 to C22, C31 to C23, C32 to C24, C37 to C25, C29 to C26, C5 to C27, C6 to C28, C40 to C29, C22 to C3, C21 to C30, C24 to C31, C28 to C32, C41 to C34, C30 to C35, C1 to C36, C34 to C37, C2 to C38, C25 to C39, C23 to C4, C27 to C40, C9 to C41, C26 to C5, C35 to C6, C36 to C7, C38 to C8, C39 to C9, D4 to D1, D1 to D3, D3 to D4, J2 to J1, J1 to J2, J4 to J3, L3 to L1, L4 to L2, L1 to L3, L7 to L4, L6 to L5, R6 to R1, R7 to R2, R11 to R3, R9 to R4, R10 to R5, R12 to R6, R4 to R7, R5 to R8, R8 to R9, U2 to U1, U3 to U2, U7 to U3, U5 to U4, U4 to U5, U8 to U7, U1 to U8, Y2 to Y1, Y1 to Y2

Commit message: SchChanges&fixLabels
Parts:
- moved C20 0.18 mm to (135.3, 115.1)
- moved C21 0.18 mm to (132.9, 117.8)
- moved Y1 0.18 mm to (135.9, 117.6)
- moved U8 0.07 mm to (142.6, 115.2)
- renumbered BOOT to BOOT1, RESET to RESET1, RESET_CC to RESET_CC1, SW to SW1
Connections:
- U8 pad 12: /LED4 -> Net-(U8-Pad12)
- U8 pad 37: Net-(U8-Pad37) -> /LED4

Commit message: newFloorPlanInProgress
Parts:
- moved C18 60.6 mm to (148.2, 158.3), turned to 0 degrees
- moved C19 60.3 mm to (148.2, 156.8), turned to 0 degrees
- moved C13 56.7 mm to (135.0, 163.6), turned to 180 degrees
- moved C14 55.5 mm to (135.0, 162.0), turned to 180 degrees
- moved C20 53.1 mm to (140.8, 167.9), turned to 225 degrees
- moved C17 52.8 mm to (139.2, 155.7), turned to 135 degrees
- moved C15 52.7 mm to (137.1, 157.8), turned to 135 degrees
- moved C16 52.7 mm to (138.1, 156.7), turned to 135 degrees
- moved C29 50.0 mm to (152.3, 164.7)
- moved Y2 49.9 mm to (149.8, 162.1)
- moved C36 49.9 mm to (152.3, 163.1)
- moved C25 49.8 mm to (152.3, 166.3)
- moved C21 49.7 mm to (136.4, 167.4), turned to 315 degrees
- moved C38 49.5 mm to (152.2, 161.2)
- moved Y1 48.5 mm to (138.6, 166.0), turned to 135 degrees
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- renumbered BOOT1 to BOOT, RESET1 to RESET, RESET_CC1 to RESET_CC, SW1 to SW

Commit message: NewFloorPlan
Parts:
- moved C18 56.8 mm to (128.6, 105.1)
- moved C36 56.1 mm to (132.1, 110.7), turned to 90 degrees
- moved C29 55.4 mm to (136.0, 111.7), turned to 0 degrees
- moved Y2 55.1 mm to (130.5, 110.5)
- moved C19 53.9 mm to (128.6, 106.6)
- moved C38 53.8 mm to (133.6, 110.7), turned to 270 degrees
- moved C25 53.8 mm to (146.0, 112.9)
- moved C15 53.5 mm to (125.7, 105.5), turned to 90 degrees
- moved C16 53.1 mm to (124.2, 105.5), turned to 90 degrees
- moved C13 53.0 mm to (119.4, 113.0)
- moved C14 52.9 mm to (119.4, 111.5)
- moved U4 52.9 mm to (138.0, 112.8)
- moved C17 52.8 mm to (122.7, 105.5), turned to 90 degrees
- moved U8 52.5 mm to (125.3, 111.6), turned to 180 degrees
- moved C20 52.1 mm to (127.2, 117.6), turned to 270 degrees
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- renumbered SW to SW1
Connections:
- net /RF_N_2_4_GHZ renamed /2_4_GHZ_RF_N
- net /RF_N_SUB_1_GHZ renamed /SUB_1_GHZ_RF_N
- net /RF_P_2_4_GHZ renamed /2_4_GHZ_RF_P
- net /RF_P_SUB_1_GHZ renamed /SUB_1_GHZ_RF_P
Other:
- board size 80 x 20 mm -> 81 x 20 mm

Commit message: updated floorplan
Parts:
- removed BOOT, RESET_CC: SW, CatSniffer:TS1088R02026
- added BOOT1: SW, CatSniffer:TS1088R02026, F.Cu at (114.6, 117.5)
- added RESET_CC1: SW, CatSniffer:TS1088R02026, F.Cu at (107.1, 117.5)
- L1, L2, L3, L4, L5: footprint Inductor_SMD:L_0603_1608Metric_Pad1.05x0.95mm_HandSolder -> Inductor_SMD:L_0603_1608Metric
- R1, R2, R3, R4, R5, R6, R7, R8, R9: footprint Resistor_SMD:R_0603_1608Metric_Pad0.98x0.95mm_HandSolder -> Resistor_SMD:R_0603_1608Metric
- Y2: footprint Crystal:Crystal_SMD_2012-2Pin_2.0x1.2mm_HandSoldering -> Crystal:Crystal_SMD_2012-2Pin_2.0x1.2mm
- moved JP1 32.3 mm to (129.7, 101.3), turned to 180 degrees
- moved C34 24.9 mm to (133.5, 117.9)
- moved R6 23.8 mm to (135.0, 117.9), turned to 90 degrees
- moved C21 19.4 mm to (140.8, 118.0)
- moved C26 19.4 mm to (124.7, 113.2), turned to 315 degrees
- moved J3 19.4 mm to (126.5, 116.5)
- moved Y1 19.3 mm to (143.7, 117.9)
- moved C20 19.2 mm to (146.5, 117.8)
- moved C13 19.2 mm to (137.9, 118.0), turned to 270 degrees
- moved C23 18.9 mm to (125.3, 102.7), turned to 135 degrees
- moved C39 18.7 mm to (120.9, 104.2), turned to 225 degrees
- moved C19 17.6 mm to (146.2, 106.5)
- moved C36 17.5 mm to (149.6, 108.8)
- moved C16 17.5 mm to (136.4, 118.0), turned to 270 degrees
- moved Y2 17.1 mm to (147.5, 109.3), turned to 180 degrees
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- renumbered RESET to RESET1
Routing:
- net /VDDS: track 0.00 -> 18.4 mm
- net GND: track 0.00 -> 16.2 mm, vias 0 -> 2
- net Net-(C6-Pad2): track 0.00 -> 11.3 mm
- net /VDDR: track 0.00 -> 8.99 mm
- net /X48M_N: track 0.00 -> 7.70 mm
- net Net-(C36-Pad1): track 0.00 -> 7.45 mm
- net Net-(C7-Pad2): track 0.00 -> 7.25 mm
- net Net-(C38-Pad1): track 0.00 -> 5.66 mm
- net /X48M_P: track 0.00 -> 5.42 mm
- net +3V3: track 0.00 -> 5.28 mm
- net /RFO: track 0.00 -> 5.23 mm
- net /RFI_P: track 0.00 -> 5.17 mm
- net /RFI_N: track 0.00 -> 5.17 mm
- net /SW_RFO: track 0.00 -> 4.55 mm
- net Net-(C8-Pad2): track 0.00 -> 4.28 mm
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Other:
- rule trace_min: 0.2 -> 0.15
