File: hardware/CatSniffer.sch (KiCad schematic (older format))
At the start: 76 parts, among them J1 Antenna, J2 Conn_01x06_Female, J3 Conn_01x06_Female, P1 USB_C_Plug_USB2.0, SW1 SW, U1 AP2112K-3.3, U2 RFSW8006QTR7, U3 ATSAMD21E18A, U4 0900PC15A0036, U5 0900FM15D0039, U6 SW409, U7 SX1262IMLTRT, U8 CC1352R1F3RGZR, Y1 48MHz, Y2 32.768kHz, Y3 32Mhz

Commit message: rename project kicad
Parts:
- BOOT1, RESET1, RESET_CC1, SW1: symbol CatStick-rescue:SW_Push-Switch -> CatSniffer-rescue:SW_Push-Switch-CatStick-rescue
- C1, C10, C11, C12, C13, C14, C15, C16, C17, C18, C19, C2, C20, C23, C25, C26, C27, C28, C30, C32, C34, C36, C37, C6, C7, C8, C9: symbol CatStick-rescue:C-Device -> CatSniffer-rescue:C-Device-CatStick-rescue
- C21, C22, C24, C29, C3, C31, C33, C35, C4, C5: symbol CatStick-rescue:C_Small-Device -> CatSniffer-rescue:C_Small-Device-CatStick-rescue
- D1, D2, D3, D4: symbol CatStick-rescue:LED_Small-Device -> CatSniffer-rescue:LED_Small-Device-CatStick-rescue
- F1: symbol CatStick-rescue:Fuse_Small-Device -> CatSniffer-rescue:Fuse_Small-Device-CatStick-rescue
- J1: symbol CatStick-rescue:Conn_Coaxial-Connector -> CatSniffer-rescue:Conn_Coaxial-Connector-CatStick-rescue
- J2, J3: symbol CatStick-rescue:Conn_01x06_Female-Connector -> CatSniffer-rescue:Conn_01x06_Female-Connector-CatStick-rescue
- JP1: symbol CatStick-rescue:Jumper_3_Bridged12-Jumper -> CatSniffer-rescue:Jumper_3_Bridged12-Jumper-CatStick-rescue
- L1: symbol CatStick-rescue:Ferrite_Bead-Device -> CatSniffer-rescue:Ferrite_Bead-Device-CatStick-rescue
- L2, L3: symbol CatStick-rescue:L-Device -> CatSniffer-rescue:L-Device-CatStick-rescue
- L4, L5: symbol CatStick-rescue:L_Small-Device -> CatSniffer-rescue:L_Small-Device-CatStick-rescue
- P1: symbol CatStick-rescue:USB_C_Plug_USB2.0-Connector -> CatSniffer-rescue:USB_C_Plug_USB2.0-Connector-CatStick-rescue
- R1, R2, R3, R4, R5, R7, R8, R9: symbol CatStick-rescue:R_Small-Device -> CatSniffer-rescue:R_Small-Device-CatStick-rescue
- R6: symbol CatStick-rescue:R-Device -> CatSniffer-rescue:R-Device-CatStick-rescue
- U1: symbol CatStick-rescue:AP2112K-1.2-Regulator_Linear-CatStick-rescue -> CatSniffer-rescue:AP2112K-1.2-Regulator_Linear-CatStick-rescue-CatStick-rescue
- U2: symbol CatStick-rescue:RFSW8006QTR7-electroniccats -> CatSniffer-rescue:RFSW8006QTR7-electroniccats-CatStick-rescue
- U3: symbol CatStick-rescue:ATSAMD21E18A-electroniccats -> CatSniffer-rescue:ATSAMD21E18A-electroniccats-CatStick-rescue
- U4: symbol CatStick-rescue:0900PC15A0036-Electronic_Cats -> CatSniffer-rescue:0900PC15A0036-Electronic_Cats-CatStick-rescue
- U5: symbol CatStick-rescue:0900FM15D0039-Electronic_Cats -> CatSniffer-rescue:0900FM15D0039-Electronic_Cats-CatStick-rescue
- U6: symbol CatStick-rescue:MASWSS0115-RF_Switch -> CatSniffer-rescue:MASWSS0115-RF_Switch-CatStick-rescue
- U8: symbol CatStick-rescue:CC1352R1F3RGZR-cc1352-cc1352-swim-thermo-rescue-CatStick-rescue -> CatSniffer-rescue:CC1352R1F3RGZR-cc1352-cc1352-swim-thermo-rescue-CatStick-rescue-CatStick-rescue
- Y1, Y3: symbol CatStick-rescue:Crystal_GND24-Device -> CatSniffer-rescue:Crystal_GND24-Device-CatStick-rescue
- Y2: symbol CatStick-rescue:Crystal-Device -> CatSniffer-rescue:Crystal-Device-CatStick-rescue

Commit message: ChngCC1352P
Parts:
- removed U8: CC1352R1F3RGZR, Package_DFN_QFN:VQFN-48-1EP_7x7mm_P0.5mm_EP5.15x5.15mm_ThermalVias, symbol CatSniffer-rescue:CC1352R1F3RGZR-cc1352-cc1352-swim-thermo-rescue-CatStick-resc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
- added U8: CC1352P1F3RGZT, Package_DFN_QFN:VQFN-48-1EP_7x7mm_P0.5mm_EP5.15x5.15mm_ThermalVias, symbol CC1352P1F3RGZT:CC1352P1F3RGZT
- BOOT1, RESET1, RESET_CC1, SW1: symbol CatSniffer-rescue:SW_Push-Switch-CatStick-rescue -> CatSniffer-rescue:SW_Push-Switch-CatStick-rescue-CatSniffer-rescue
- C1, C10, C11, C12, C13, C14, C15, C16, C17, C18, C19, C2, C20, C23, C25, C26, C27, C28, C30, C32, C34, C36, C37, C6, C7, C8, C9: symbol CatSniffer-rescue:C-Device-CatStick-rescue -> CatSniffer-rescue:C-Device-CatStick-rescue-CatSniffer-rescue
- C21, C22, C24, C29, C3, C31, C33, C35, C4, C5: symbol CatSniffer-rescue:C_Small-Device-CatStick-rescue -> CatSniffer-rescue:C_Small-Device-CatStick-rescue-CatSniffer-rescue
- D1, D2, D3, D4: symbol CatSniffer-rescue:LED_Small-Device-CatStick-rescue -> CatSniffer-rescue:LED_Small-Device-CatStick-rescue-CatSniffer-rescue
- F1: symbol CatSniffer-rescue:Fuse_Small-Device-CatStick-rescue -> CatSniffer-rescue:Fuse_Small-Device-CatStick-rescue-CatSniffer-rescue
- J1: symbol CatSniffer-rescue:Conn_Coaxial-Connector-CatStick-rescue -> CatSniffer-rescue:Conn_Coaxial-Connector-CatStick-rescue-CatSniffer-rescue
- J2, J3: symbol CatSniffer-rescue:Conn_01x06_Female-Connector-CatStick-rescue -> CatSniffer-rescue:Conn_01x06_Female-Connector-CatStick-rescue-CatSniffer-rescue
- JP1: symbol CatSniffer-rescue:Jumper_3_Bridged12-Jumper-CatStick-rescue -> CatSniffer-rescue:Jumper_3_Bridged12-Jumper-CatStick-rescue-CatSniffer-rescue
- L1: symbol CatSniffer-rescue:Ferrite_Bead-Device-CatStick-rescue -> CatSniffer-rescue:Ferrite_Bead-Device-CatStick-rescue-CatSniffer-rescue
- L2, L3: symbol CatSniffer-rescue:L-Device-CatStick-rescue -> CatSniffer-rescue:L-Device-CatStick-rescue-CatSniffer-rescue
- L4, L5: symbol CatSniffer-rescue:L_Small-Device-CatStick-rescue -> CatSniffer-rescue:L_Small-Device-CatStick-rescue-CatSniffer-rescue
- P1: symbol CatSniffer-rescue:USB_C_Plug_USB2.0-Connector-CatStick-rescue -> CatSniffer-rescue:USB_C_Plug_USB2.0-Connector-CatStick-rescue-CatSniffer-rescue
- R1, R2, R3, R4, R5, R7, R8, R9: symbol CatSniffer-rescue:R_Small-Device-CatStick-rescue -> CatSniffer-rescue:R_Small-Device-CatStick-rescue-CatSniffer-rescue
- R6: symbol CatSniffer-rescue:R-Device-CatStick-rescue -> CatSniffer-rescue:R-Device-CatStick-rescue-CatSniffer-rescue
- U1: symbol CatSniffer-rescue:AP2112K-1.2-Regulator_Linear-CatStick-rescue-CatStick-rescue -> CatSniffer-rescue:AP2112K-1.2-Regulator_Linear-CatStick-rescue-CatStick-rescue-CatSniffer-rescue
- U2: symbol CatSniffer-rescue:RFSW8006QTR7-electroniccats-CatStick-rescue -> CatSniffer-rescue:RFSW8006QTR7-electroniccats-CatStick-rescue-CatSniffer-rescue
- U3: symbol CatSniffer-rescue:ATSAMD21E18A-electroniccats-CatStick-rescue -> CatSniffer-rescue:ATSAMD21E18A-electroniccats-CatStick-rescue-CatSniffer-rescue
- U4: symbol CatSniffer-rescue:0900PC15A0036-Electronic_Cats-CatStick-rescue -> CatSniffer-rescue:0900PC15A0036-Electronic_Cats-CatStick-rescue-CatSniffer-rescue
- U5: symbol CatSniffer-rescue:0900FM15D0039-Electronic_Cats-CatStick-rescue -> CatSniffer-rescue:0900FM15D0039-Electronic_Cats-CatStick-rescue-CatSniffer-rescue
- U6: symbol CatSniffer-rescue:MASWSS0115-RF_Switch-CatStick-rescue -> CatSniffer-rescue:MASWSS0115-RF_Switch-CatStick-rescue-CatSniffer-rescue
- Y1, Y3: symbol CatSniffer-rescue:Crystal_GND24-Device-CatStick-rescue -> CatSniffer-rescue:Crystal_GND24-Device-CatStick-rescue-CatSniffer-rescue
- Y2: symbol CatSniffer-rescue:Crystal-Device-CatStick-rescue -> CatSniffer-rescue:Crystal-Device-CatStick-rescue-CatSniffer-rescue
Connections:
- net 2_4_GHZ_RF_N: now also U8.2 (RF_N_2_4GHZ)
- net 2_4_GHZ_RF_P: now also U8.1 (RF_P_2_4GHZ)
- net BOOT: now also U8.21 (DIO_15)
- net DCDC_SW: now also U8.33 (DCDC_SW)
- net GND: now also U8.49 (EGP), U8.49_1 (EGP), U8.49_10 (EGP), U8.49_11 (EGP), U8.49_12 (EGP), U8.49_13 (EGP), U8.49_14 (EGP), U8.49_15 (EGP), U8.49_16 (EGP), U8.49_17 (EGP), U8.49_18 (EGP), U8.49_19 (EGP), U8.49_2 (EGP), U8.49_20 (EGP), U8.49_21 (EGP), U8.49_3 (EGP), U8.49_4 (EGP), U8.49_5 (EGP), U8.49_6 (EGP), U8.49_7 (EGP), U8.49_8 (EGP), U8.49_9 (EGP)
- net LED4: now also U8.37 (DIO_24)
- net RESET_CC: now also U8.35 (~RESET_N)
- net RXD: now also U8.19 (DIO_13)
- net RX_TX: now also U8.7 (RX_TX)
- net SUB_1_GHZ_RF_N: now also U8.4 (RF_N_SUB_1GHZ)
- net SUB_1_GHZ_RF_P: now also U8.3 (RF_P_SUB_1GHZ)
- net TXD: now also U8.18 (DIO_12)
- net VDDR: now also U8.45 (VDDR), U8.48 (VDDR_RF)
- net VDDS: now also U8.13 (VDDS2), U8.22 (VDDS3), U8.34 (VDDS_DCDC), U8.44 (VDDS)
- net X48M_N: now also U8.46 (X48M_N)
- net X48M_P: now also U8.47 (X48M_P)
- net cJTAG_TCK: now also U8.25 (JTAG_TCKC)
- net cJTAG_TMSC: now also U8.24 (JTAG_TMSC)
- net at C34.1, Y2.1: now also U8.8 (X32K_Q1)
- net at C36.1, Y2.2: now also U8.9 (X32K_Q2)
- net at C37.1: now also U8.23 (DCOUPL)
- no-connect marks 27 -> 26
Other:
- moved on the sheet: C18, C19, C32, C34, C36, C37, D4, R6, R9, Y1, Y2
