File: hardware/CatSniffer.kicad_sch (KiCad schematic)
At the start: 91 parts, among them J1 Antenna, J2 Conn_01x06_Female, J3 Conn_01x06_Female, P1 USB_C_Plug_USB2.0, SW1 SW, U1 AP2112K-3.3, U2 RFSW8006QTR7, U3 RP2040, U4 0900PC15A0036, U5 0900FM15D0039, U6 PE42421, U7 SX1262IMLTRT, U8 CC1352P1F3RGZT, U9 W25Q16JV, Y1 48MHz, Y2 32.768kHz, Y3 32Mhz, Y4 12MHz

Commit message: Initial routing
Parts:
- removed Y4: 12MHz, Crystal:Crystal_SMD_5032-2Pin_5.0x3.2mm, symbol Device:Crystal_Small
- added Y4: 12MHz, Crystal:Crystal_SMD_3225-4Pin_3.2x2.5mm, symbol Device:Crystal_GND23_Small
Connections:
- net JTAG/TCK is gone; now on net cJTAG_TCK: U3.14 (GPIO11)
- net GND: now also Y4.2, Y4.4
- net SWCLK: no longer U3.24 (SWCLK)
- net SWDIO: no longer U3.25 (SWD)
- net at C28.1, R12.1: now also Y4.3
- net at C4.1, U3.20 (XIN): now also Y4.1
- no-connect marks 28 -> 30
Changed lines of the file:
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@@
   (no_connect (at 71.12 219.71))
   (no_connect (at 71.12 201.93))
+  (no_connect (at 313.69 97.79))
+  (no_connect (at 313.69 95.25))
   (no_connect (at 116.84 201.93))
   (no_connect (at 116.84 217.17))
@@
     (stroke (width 0) (type default) (color 0 0 0 0))
   )
-  (wire (pts (xy 311.15 95.25) (xy 313.69 95.25))
-    (stroke (width 0) (type default) (color 0 0 0 0))
-  )
   (polyline (pts (xy 12.065 84.963) (xy 272.796 84.963))
     (stroke (width 0) (type default) (color 0 0 0 0))
@@
     (stroke (width 0) (type default) (color 0 0 0 0))
   )
-  (wire (pts (xy 285.75 92.71) (xy 285.75 93.98))
+  (wire (pts (xy 285.75 92.71) (xy 285.75 95.25))
     (stroke (width 0) (type default) (color 0 0 0 0))
   )
@@
     (stroke (width 0) (type default) (color 0 0 0 0))
   )
-  (wire (pts (xy 295.91 92.71) (xy 295.91 93.98))
+  (wire (pts (xy 295.91 92.71) (xy 295.91 95.25))
     (stroke (width 0) (type default) (color 0 0 0 0))
   )
@@
     (stroke (width 0) (type default) (color 0 0 0 0))
   )
+  (wire (pts (xy 290.83 82.55) (xy 290.83 83.82))
+    (stroke (width 0) (type default) (color 0 0 0 0))
+  )
   (wire (pts (xy 35.56 154.94) (xy 36.83 154.94))
     (stroke (width 0) (type default) (color 0 0 0 0))
@@
     (stroke (width 0) (type default) (color 0 0 0 0))
   )
+  (wire (pts (xy 290.83 88.9) (xy 290.83 90.17))
+    (stroke (width 0) (type default) (color 0 0 0 0))
+  )
   (wire (pts (xy 464.566 224.79) (xy 464.566 229.108))
     (stroke (width 0) (type default) (color 0 0 0 0))
@@
     (stroke (width 0) (type default) (color 0 0 0 0))
   )
-  (wire (pts (xy 311.15 97.79) (xy 313.69 97.79))
-    (stroke (width 0) (type default) (color 0 0 0 0))
-  )
   (wire (pts (xy 314.198 197.104) (xy 312.039 197.104))
     (stroke (width 0) (type default) (color 0 0 0 0))
@@
     (effects (font (size 1.27 1.27)) (justify left bottom))
   )
-  (label "JTAG{slash}TCK" (at 369.57 57.15 0)
+  (label "cJTAG_TCK" (at 369.57 57.15 0)
     (effects (font (size 1.27 1.27)) (justify left bottom))
   )
@@
     (pin "1")
   )
-  (symbol (lib_id "power:GND") (at 285.75 93.98 0) (unit 1)
+  (symbol (lib_id "power:GND") (at 285.75 95.25 0) (unit 1)
     (in_bom yes) (on_board yes)
-    (property "Reference" "#PWR018" (id 0) (at 285.75 100.33 0)
+    (property "Reference" "#PWR018" (id 0) (at 285.75 101.6 0)
       (effects (font (size 1.27 1.27)) hide)
     )
-    (property "Value" "GND" (id 1) (at 285.75 97.79 0))
-    (property "Footprint" "" (id 2) (at 285.75 93.98 0)
+    (property "Value" "GND" (id 1) (at 285.75 99.06 0))
+    (property "Footprint" "" (id 2) (at 285.75 95.25 0)
       (effects (font (size 1.27 1.27)) hide)
     )
-    (property "Datasheet" "" (id 3) (at 285.75 93.98 0)
+    (property "Datasheet" "" (id 3) (at 285.75 95.25 0)
       (effects (font (size 1.27 1.27)) hide)
     )
@@
     (pin "1")
   )
-  (symbol (lib_id "Device:Crystal_Small") (at 290.83 86.36 0) (unit 1)
-    (in_bom yes) (on_board yes) (fields_autoplaced)
-    (property "Reference" "Y4" (id 0) (at 290.83 80.01 0))
-    (property "Value" "12MHz" (id 1) (at 290.83 82.55 0))
-    (property "Footprint" "Crystal:Crystal_SMD_5032-2Pin_5.0x3.2mm" (id 2) (at 290.83 86.36 0)
-      (effects (font (size 1.27 1.27)) hide)
-    )
-    (property "Datasheet" "~" (id 3) (at 290.83 86.36 0)
-      (effects (font (size 1.27 1.27)) hide)
-    )
-    (property "LCSC#" "C709001" (id 4) (at 290.83 86.36 0)
-      (effects (font (size 1.27 1.27)) hide)
-    )
-    (property "manf#" "CM4012M00020T8188026" (id 5) (at 290.83 86.36 0)
-      (effects (font (size 1.27 1.27)) hide)
-    )
-    (property "provedor" "LCSC" (id 6) (at 290.83 86.36 0)
-      (effects (font (size 1.27 1.27)) hide)
-    )
-    (pin "1")
-    (pin "2")
-  )
   (symbol (lib_id "power:+1V2") (at 334.01 19.05 0) (unit 1)
     (in_bom yes) (on_board yes) (fields_autoplaced)
@@
     (pin "1")
   )
+  (symbol (lib_id "power:GND") (at 290.83 90.17 0) (unit 1)
+    (in_bom yes) (on_board yes)
+    (property "Reference" "#PWR0104" (id 0) (at 290.83 96.52 0)
+      (effects (font (size 1.27 1.27)) hide)
+    )
+    (property "Value" "GND" (id 1) (at 290.83 93.98 0))
+    (property "Footprint" "" (id 2) (at 290.83 90.17 0)
+      (effects (font (size 1.27 1.27)) hide)
+    )
+    (property "Datasheet" "" (id 3) (at 290.83 90.17 0)
+      (effects (font (size 1.27 1.27)) hide)
+    )
+    (pin "1")
+  )
   (symbol (lib_id "power:GND") (at 330.2 135.89 0) (unit 1)
     (in_bom yes) (on_board yes)
@@
     (pin "1")
   )
+  (symbol (lib_id "Device:Crystal_GND23_Small") (at 290.83 86.36 0) (unit 1)
+    (in_bom yes) (on_board yes)
+    (property "Reference" "Y4" (id 0) (at 295.91 81.28 0))
+    (property "Value" "12MHz" (id 1) (at 297.18 83.82 0))
+    (property "Footprint" "Crystal:Crystal_SMD_3225-4Pin_3.2x2.5mm" (id 2) (at 290.83 86.36 0)
+      (effects (font (size 1.27 1.27)) hide)
+    )
+    (property "Datasheet" "~" (id 3) (at 290.83 86.36 0)
+      (effects (font (size 1.27 1.27)) hide)
+    )
+    (property "LCSC#" "C521581" (id 4) (at 290.83 86.36 0)
+      (effects (font (size 1.27 1.27)) hide)
+    )
+    (property "manf#" "XXHBBCNANF-12.000000MHZ" (id 5) (at 290.83 86.36 0)
+      (effects (font (size 1.27 1.27)) hide)
+    )
+    (property "provedor" "LCSC" (id 6) (at 290.83 86.36 0)
+      (effects (font (size 1.27 1.27)) hide)
+    )
+    (pin "1")
+    (pin "2")
+    (pin "3")
+    (pin "4")
+  )
   (symbol (lib_id "power:GND") (at 391.16 135.89 0) (unit 1)
     (in_bom yes) (on_board yes)
@@
     (pin "1")
   )
-  (symbol (lib_id "power:GND") (at 295.91 93.98 0) (unit 1)
+  (symbol (lib_id "power:GND") (at 295.91 95.25 0) (unit 1)
     (in_bom yes) (on_board yes)
-    (property "Reference" "#PWR065" (id 0) (at 295.91 100.33 0)
+    (property "Reference" "#PWR065" (id 0) (at 295.91 101.6 0)
       (effects (font (size 1.27 1.27)) hide)
     )
-    (property "Value" "GND" (id 1) (at 295.91 97.79 0))
-    (property "Footprint" "" (id 2) (at 295.91 93.98 0)
+    (property "Value" "GND" (id 1) (at 295.91 99.06 0))
+    (property "Footprint" "" (id 2) (at 295.91 95.25 0)
       (effects (font (size 1.27 1.27)) hide)
     )
-    (property "Datasheet" "" (id 3) (at 295.91 93.98 0)
+    (property "Datasheet" "" (id 3) (at 295.91 95.25 0)
       (effects (font (size 1.27 1.27)) hide)
     )
@@
     (pin "2")
   )
+  (symbol (lib_id "power:GND") (at 290.83 82.55 180) (unit 1)
+    (in_bom yes) (on_board yes)
+    (property "Reference" "#PWR0103" (id 0) (at 290.83 76.2 0)
+      (effects (font (size 1.27 1.27)) hide)
+    )
+    (property "Value" "GND" (id 1) (at 290.83 78.74 0))
+    (property "Footprint" "" (id 2) (at 290.83 82.55 0)
+      (effects (font (size 1.27 1.27)) hide)
+    )
+    (property "Datasheet" "" (id 3) (at 290.83 82.55 0)
+      (effects (font (size 1.27 1.27)) hide)
+    )
+    (pin "1")
+  )
   (sheet_instances
     (path "/" (page "1"))
@@
       (reference "#PWR0102") (unit 1) (value "GND") (footprint "")
     )
+    (path "/fb4eda9e-2267-4024-9c32-60469c5c5602"
+      (reference "#PWR0103") (unit 1) (value "GND") (footprint "")
+    )
+    (path "/6bbe5852-16fd-4d82-bbb8-634ae446ffff"
+      (reference "#PWR0104") (unit 1) (value "GND") (footprint "")
+    )
     (path "/00000000-0000-0000-0000-000060c2b98f"
       (reference "BOOT1") (unit 1) (value "SW") (footprint "CatSniffer:TS1088R02026")
@@
       (reference "Y3") (unit 1) (value "32Mhz") (footprint "Crystal:Crystal_SMD_2520-4Pin_2.5x2.0mm")
     )
-    (path "/2ce791c0-a4fd-4dc9-a0a5-6c30852e2179"
-      (reference "Y4") (unit 1) (value "12MHz") (footprint "Crystal:Crystal_SMD_5032-2Pin_5.0x3.2mm")
+    (path "/8640b6bd-3a85-4e04-bfcd-a54fc955be99"
+      (reference "Y4") (unit 1) (value "12MHz") (footprint "Crystal:Crystal_SMD_3225-4Pin_3.2x2.5mm")
     )
   )
