File: hardware/CatSniffer.kicad_sch (KiCad schematic)
At the start: 91 parts, among them J1 Antenna, J2 Conn_01x06_Female, J3 Conn_01x06_Female, P1 USB_C_Plug_USB2.0, SW1 SW, U1 AP2112K-3.3, U2 RFSW8006QTR7, U3 RP2040, U4 0900PC15A0036, U5 0900FM15D0039, U6 PE42421, U7 SX1262IMLTRT, U8 CC1352P1F3RGZT, U9 W25Q16JV, Y1 48MHz, Y2 32.768kHz, Y3 32Mhz, Y4 12MHz

Commit message: fix(Hw):Update_DNP_Parts
Parts:
- removed J2: Conn_01x06_Female, Connector:Tag-Connect_TC2030-IDC-NL_2x03_P1.27mm_Vertical, symbol CatSniffer-rescue:Conn_01x06_Female-Connector-CatStick-rescue-CatSniffer-rescue
- J3, JP1: now not fitted
Connections:
- no-connect marks 36 -> 30
Other:
- note removed: "SWD FOR RP2040"

Commit message: feat(HW):CC1352P74T0RGZR_Updated
Parts:
- L1: value BLM18HE152SN1D -> BLM18HE152SN1D
- U8: value CC1352P1F3RGZT -> CC1352P74T0RGZR; manf# CC1352P1F3RGZT -> CC1352P74T0RGZR
