File: hardware/M.2/M.2.kicad_pcb (KiCad board)
At the start: 2 copper layers, 81 x 20 mm, 65 parts, among them J1 Antenna, J3 Conn_01x06_Female, SW1 SW, U1 AP2112K-3.3, U2 RFSW8006QTR7, U3 RP2040, U4 0900PC15A0036, U8 CC1352P1F3RGZT, U9 W25Q16JV, Y1 48MHz, Y2 32.768kHz, Y4 12MHz

Commit message: feat(Hw):Update_Floorplan
Parts:
- removed C1: 1uF, Capacitor_SMD:C_0603_1608Metric
- removed C2: 0.1uF, Capacitor_SMD:C_0603_1608Metric
- removed U1: AP2112K-3.3, Package_TO_SOT_SMD:SOT-23-5
- added J2: M.2 B, Footprints:M.2_Key_B_Fingers, F.Cu at (116.8, 59.1)
- moved RESET_CC1 59.0 mm to (155.8, 46.7)
- moved D1 58.9 mm to (160.0, 56.9)
- moved D2 58.9 mm to (160.0, 55.4)
- moved D3 58.9 mm to (160.0, 53.8)
- moved D4 58.9 mm to (160.0, 58.5)
- moved R3 58.9 mm to (156.8, 56.9)
- moved R5 58.9 mm to (156.8, 53.8)
- moved R4 58.9 mm to (156.8, 55.4)
- moved R9 58.9 mm to (156.8, 58.5)
- moved BOOT1 57.6 mm to (163.7, 46.8)
- moved C30 35.8 mm to (143.8, 51.5)
- moved C38 35.8 mm to (132.5, 50.1)
- moved C40 35.8 mm to (134.2, 50.1)
- moved C41 35.8 mm to (131.3, 53.5)
- moved C42 35.8 mm to (128.4, 51.6)
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Routing:
- net /VDDR: track 2.18 -> 0.00 mm, vias 1 -> 0
- net /LED4: track 2.16 -> 0.00 mm, vias 1 -> 0
- net Net-(D3-K): track 1.52 -> 0.00 mm
- net Net-(D4-K): track 1.51 -> 0.00 mm
- net Net-(D2-K): track 1.51 -> 0.00 mm
- net Net-(D1-K): track 1.51 -> 0.00 mm
- net /LED1: track 1.42 -> 0.00 mm, vias 1 -> 0
- net /LED2: track 1.38 -> 0.00 mm, vias 1 -> 0
- net /LED3: track 1.26 -> 0.00 mm, vias 1 -> 0
- removed copper zone on B.Cu, net GND
- removed copper zone on F.Cu, net GND
Other:
- board size 81 x 20 mm -> 52 x 30 mm
- board text removed: "CatSniffer V3.2"
- board text removed: "CatSniffer v3.2"
- board text removed: "electroniccats.com"
- board text removed: "pwnlab.com.mx"
