File: hardware/M.2/M.2.kicad_sch (KiCad schematic)
At the start: 65 parts, among them J1 Antenna, J3 Conn_01x06_Female, SW1 SW, U1 AP2112K-3.3, U2 RFSW8006QTR7, U3 RP2040, U4 0900PC15A0036, U8 CC1352P1F3RGZT, U9 W25Q16JV, Y1 48MHz, Y2 32.768kHz, Y4 12MHz

Commit message: feat(Hw):Update_Floorplan
Parts:
- removed C1: 1uF, Capacitor_SMD:C_0603_1608Metric, symbol CatSniffer-rescue:C-Device-CatStick-rescue-CatSniffer-rescue
- removed C2: 0.1uF, Capacitor_SMD:C_0603_1608Metric, symbol CatSniffer-rescue:C-Device-CatStick-rescue-CatSniffer-rescue
- removed U1: AP2112K-3.3, Package_TO_SOT_SMD:SOT-23-5, symbol CatSniffer-rescue:AP2112K-1.2-Regulator_Linear-CatStick-rescue-CatStick-rescue-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
- added J2: M.2 B, Footprints:M.2_Key_B_Fingers, symbol Connector_Generic:Conn_2Rows-75Pins
Other:
- note removed: "REGULATOR AND BATTERY"
